File: src/HardwareDesign/Rev0.1.0/PDNode-600 Pro.brd (EAGLE design)
At the start: 245 x 100 mm, 652 parts, among them IC1 AP22653W6, IC11 STUSB4710, IC12 TPS552882, IC13 INA219BIDCNT, IC14 STUSB4710, IC15 TPS552882, IC16 INA219BIDCNT, IC17 STUSB4710, IC18 TPS552882, IC19 INA219BIDCNT, IC2 AP22653W6, IC20 STUSB4710, IC21 TPS552882, IC22 INA219BIDCNT, IC23 STUSB4710, IC24 TPS552882, IC25 INA219BIDCNT, IC26 RP2040, IC27 W25Q128JVPIQ, IC28 MCP6001R, IC29 CAT24C512HU5IGT3, IC3 AP22653W6, IC31 STUSB4710, IC32 TPS552882, IC33 INA219BIDCNT, IC34 STUSB4710, IC35 TPS552882, IC36 INA219BIDCNT, IC37 STUSB4710, IC38 TCA9548ARGER, IC39 W5500, IC4 SN74LVC1G04DBVR, IC40 MP2315S, IC41 TPS552882, IC42 MCP23017-E/ML, IC43 MP2315S, IC44 INA219BIDCNT, IC45 MP2315S, IC5 SN74LVC1G04DBVR, IC6 SN74LVC1G04DBVR, IC7 SN74LVC1G04DBVR, IC8 AP22653W6, J1 61400826021, J10 632722100213, J11 632722100213, J2 61400826021, J3 632722100213, J4 632722100213, J5 632722100213, J6 632722100213, J7 632722100213, J8 691244510006, J9 632722100213, T10 IPZ40N04S5L, T11 DMP3013SFV, T12 DMP3013SFV, T13 DMP3013SFV, T14 IPZ40N04S5L, T15 IPZ40N04S5L, T16 DMP3013SFV, T17 DMP3013SFV, T18 DMP3013SFV, T19 IPZ40N04S5L, T20 IPZ40N04S5L, T21 DMP3013SFV, T22 DMP3013SFV, T23 DMP3013SFV, T24 IPZ40N04S5L, T25 IPZ40N04S5L, T26 DMP3013SFV, T27 DMP3013SFV, T28 DMP3013SFV, T29 IPZ40N04S5L, T30 IPZ40N04S5L, T31 DMP3013SFV, T32 DMP3013SFV, T33 DMP3013SFV, T34 IPZ40N04S5L, T35 IPZ40N04S5L, T36 DMP3013SFV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

Commit message: Hardware design update
Parts:
- removed S1, S2: 430182050816, Wurth_Switch_WS-TASV:430182050816
- added BOOT, RESET: 430182050816, Wurth_Switch_WS-TASV:430182050816
- added U$1: (no value), SparkFun-Aesthetics:ROHS_LOGO_0.18_IN
- added U$2: (no value), SparkFun-Aesthetics:OSHW-LOGO-L
- moved R208 46.3 mm to (66.8, 12.3), turned to 0 degrees
- moved R217 32.8 mm to (76.6, 40.1), turned to 0 degrees
- moved R216 31.6 mm to (80.4, 40.1), turned to 0 degrees
- moved R215 31.4 mm to (84.2, 40.1), turned to 0 degrees
- moved R253 26.8 mm to (95.0, 4.73), turned to 0 degrees
- moved R252 26.7 mm to (94.5, 2.42), turned to 180 degrees
- moved IC38 23.8 mm to (80.4, 34.2), turned to 225 degrees
- moved C212 20.8 mm to (82.5, 32.2), turned to 45 degrees
- moved C213 20.0 mm to (83.1, 31.7), turned to 45 degrees
- moved C235 19.0 mm to (-46.6, 9.77), turned to 90 degrees
- moved VO3 18.2 mm to (-47.7, 5.04), turned to 90 degrees
- moved R243 18.0 mm to (-46.3, 8.75), turned to 0 degrees
- moved R241 17.4 mm to (-46.3, 7.75), turned to 0 degrees
- moved C251 17.3 mm to (76.5, 23.3), turned to 0 degrees
- moved L11 17.3 mm to (-43.2, 12.0), turned to 90 degrees
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- renumbered J1 to USBA_1-2, J10 to PORT7, J11 to PORT8, J2 to USBA_3-4, J3 to PORT2, J4 to PORT1, J5 to PORT3, J6 to PORT4, J7 to PORT5, J9 to PORT6
Connections:
- net GND: now also BOOT.2, BOOT.4, RESET.1, RESET.3; no longer S1.1, S1.3, S2.2, S2.4
- net RUN: now also RESET.2, RESET.4; no longer S1.2, S1.4
- net USB_BOOT: now also BOOT.1, BOOT.3; no longer S2.1, S2.3
Routing:
- net AGND: track 0.00 -> 916.2 mm
- net USBA1_EN: track 0.97 -> 177.4 mm, vias 0 -> 2
- net OCP4: track 20.3 -> 194.2 mm, vias 2 -> 5
- net OCP3: track 18.6 -> 192.4 mm, vias 2 -> 5
- net OCP1: track 54.6 -> 227.0 mm, vias 3 -> 6
- net USBA2_EN: track 0.00 -> 170.1 mm, vias 0 -> 2
- net USBA3_EN: track 1.21 -> 168.5 mm, vias 0 -> 2
- net TCA5_I2C_SDA: track 4.55 -> 171.8 mm, vias 0 -> 5
- net OCP2: track 82.2 -> 249.5 mm, vias 3 -> 5
- net TCA5_I2C_SCL: track 5.87 -> 168.7 mm, vias 0 -> 7
- net TCA4_I2C_SDA: track 3.46 -> 164.8 mm, vias 0 -> 5
- net TCA4_I2C_SCL: track 4.01 -> 161.2 mm, vias 0 -> 6
- net TCA3_I2C_SDA: track 2.04 -> 155.9 mm, vias 0 -> 4
- net USBA4_EN: track 1.33 -> 150.9 mm, vias 0 -> 2
- net TCA3_I2C_SCL: track 2.49 -> 148.3 mm, vias 0 -> 4
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- added copper zone on layer 15, net +24V_C
- added copper zone on layer 16, net GND
- added copper zone on layer 2, net GND
Other:
- board text added: "DvidMakesThings @2025 Wien https://github.com/DvidMakesThings"
- board text added: "PDNode-600 Pro"

Commit message: Add BOM
Parts:
- R215, R216, R217: value YC164-JR-0733RL -> 4D03WGJ0332T5E
- T10, T15, T20, T25, T30, T35, T40, T45: value IPZ40N04S5L -> IPZ40N04S5L2R8
- T14, T19, T24, T29, T34, T39, T44, T9: value IPZ40N04S5L -> IPZ40N04S5L-7R4
Routing:
- net N$19: track 0.00 -> 40.7 mm
- net N$18: track 0.00 -> 40.7 mm
- net N$17: track 0.00 -> 40.7 mm
- net N$16: track 0.00 -> 40.7 mm
Other:
- board text added: "1"
- board text added: "2"
- board text added: "3"
- board text added: "4"
