File: src/HardwareDesign/Rev0.1.0/PDNode-600 Pro.brd (EAGLE design)
At the start: 245 x 100 mm, 654 parts, among them IC1 AP22653W6, IC11 STUSB4710, IC12 TPS552882, IC13 INA219BIDCNT, IC14 STUSB4710, IC15 TPS552882, IC16 INA219BIDCNT, IC17 STUSB4710, IC18 TPS552882, IC19 INA219BIDCNT, IC2 AP22653W6, IC20 STUSB4710, IC21 TPS552882, IC22 INA219BIDCNT, IC23 STUSB4710, IC24 TPS552882, IC25 INA219BIDCNT, IC26 RP2040, IC27 W25Q128JVPIQ, IC28 MCP6001R, IC29 CAT24C512HU5IGT3, IC3 AP22653W6, IC31 STUSB4710, IC32 TPS552882, IC33 INA219BIDCNT, IC34 STUSB4710, IC35 TPS552882, IC36 INA219BIDCNT, IC37 STUSB4710, IC38 TCA9548ARGER, IC39 W5500, IC4 SN74LVC1G04DBVR, IC40 MP2315S, IC41 TPS552882, IC42 MCP23017-E/ML, IC43 MP2315S, IC44 INA219BIDCNT, IC45 MP2315S, IC5 SN74LVC1G04DBVR, IC6 SN74LVC1G04DBVR, IC7 SN74LVC1G04DBVR, IC8 AP22653W6, J8 691244510006, T10 IPZ40N04S5L2R8, T11 DMP3013SFV, T12 DMP3013SFV, T13 DMP3013SFV, T14 IPZ40N04S5L-7R4, T15 IPZ40N04S5L2R8, T16 DMP3013SFV, T17 DMP3013SFV, T18 DMP3013SFV, T19 IPZ40N04S5L-7R4, T20 IPZ40N04S5L2R8, T21 DMP3013SFV, T22 DMP3013SFV, T23 DMP3013SFV, T24 IPZ40N04S5L-7R4, T25 IPZ40N04S5L2R8, T26 DMP3013SFV, T27 DMP3013SFV, T28 DMP3013SFV, T29 IPZ40N04S5L-7R4, T30 IPZ40N04S5L2R8, T31 DMP3013SFV, T32 DMP3013SFV, T33 DMP3013SFV, T34 IPZ40N04S5L-7R4, T35 IPZ40N04S5L2R8, T36 DMP3013SFV, T37 DMP3013SFV, T38 DMP3013SFV, T39 IPZ40N04S5L-7R4, T40 IPZ40N04S5L2R8, T41 DMP3013SFV, T42 DMP3013SFV, T43 DMP3013SFV, T44 IPZ40N04S5L-7R4, T45 IPZ40N04S5L2R8, T6 DMP3013SFV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

Commit message: Hardware design update
Parts:
- removed IC31, IC34, IC37: STUSB4710, ds_ic_peripherals:QFN24
- added IC10, IC30, IC9: STUSB4710AQ1TR, ds_ic_peripherals:QFN50P300X300X55-16N
- IC1, IC2, IC3, IC8: value AP22653W6 -> AP22653W6-7
- IC11, IC14, IC17, IC20, IC23: value STUSB4710 -> STUSB4710AQ1TR; device ds_ic_peripherals:QFN24 -> ds_ic_peripherals:QFN50P300X300X55-16N
- T10, T15, T20, T25, T30, T35, T40, T45: value IPZ40N04S5L2R8 -> BSZ065N06LS5ATMA1
- T14, T19, T24, T29, T34, T39, T44, T9: value IPZ40N04S5L-7R4 -> BSZ065N06LS5ATMA1
- X1: value 12MHz -> X322512MSB4SI
- X2: value 25MHz -> X322525MOB4SI; device crystal-geyer_V1_0:3.2X2.5_KX-7 -> Wurth_Quartz Crystals & Oscillators_WE-XTAL:WE-XTAL_CFPX-180
- moved IC23 95.9 mm to (1.22, 79.3)
- moved IC20 48.1 mm to (25.2, 79.4)
- moved IC14 47.6 mm to (73.2, 79.4)
- moved IC11 47.6 mm to (97.0, 79.3)
- moved IC17 0.33 mm to (49.1, 79.2)
Connections:
- net CC1_PORT1: now also IC9.2; no longer IC11.2
- net CC1_PORT2: now also IC10.2; no longer IC14.2
- net CC1_PORT3: now also IC11.2; no longer IC23.2
- net CC1_PORT4: now also IC14.2; no longer IC20.2
- net CC1_PORT6: now also IC20.2; no longer IC31.2
- net CC1_PORT7: now also IC23.2; no longer IC34.2
- net CC1_PORT8: now also IC30.2; no longer IC37.2
- net CC2_PORT1: now also IC9.3; no longer IC11.4
- net CC2_PORT2: now also IC10.3; no longer IC14.4
- net CC2_PORT3: now also IC11.3; no longer IC23.4
- net CC2_PORT4: now also IC14.3; no longer IC20.4
- net CC2_PORT5: now also IC17.3; no longer IC17.4
- net CC2_PORT6: now also IC20.3; no longer IC31.4
- net CC2_PORT7: now also IC23.3; no longer IC34.4
- net CC2_PORT8: now also IC30.3; no longer IC37.4
- net GND: now also IC10.6, IC11.6, IC14.6, IC17.6, IC20.6, IC23.6, IC30.6, IC9.6, X2.2, X2.4; no longer IC11.10, IC11.25, IC14.10, IC14.25, IC17.10, IC17.25, IC20.10, IC20.25, IC23.10, IC23.25, IC31.10, IC31.25, IC34.10, IC34.25, IC37.10, IC37.25
- net IN1_PORT1: now also IC9.12; no longer IC11.18
- net IN1_PORT2: now also IC10.12; no longer IC14.18
- net IN1_PORT3: now also IC11.12; no longer IC23.18
- net IN1_PORT4: now also IC14.12; no longer IC20.18
- net IN1_PORT5: now also IC17.12; no longer IC17.18
- net IN1_PORT6: now also IC20.12; no longer IC31.18
- net IN1_PORT7: now also IC23.12; no longer IC34.18
- net IN1_PORT8: now also IC30.12; no longer IC37.18
- net N$106: now also IC17.11; no longer IC17.15
- net N$107: now also IC17.10; no longer IC17.14
- net N$108: now also IC17.7; no longer IC17.11
- net N$109: now also IC17.8; no longer IC17.12
- net N$110: now also IC17.15; no longer IC17.21
- net N$111: now also IC17.16; no longer IC17.23
- net N$112: now also IC17.9; no longer IC17.13
- net N$114: now also IC17.13; no longer IC17.19
- net N$117: now also IC17.14; no longer IC17.20
- net N$135: now also IC14.11; no longer IC20.15
- net N$136: now also IC14.10; no longer IC20.14
- net N$137: now also IC14.7; no longer IC20.11
- net N$138: now also IC14.8; no longer IC20.12
- net N$139: now also IC14.15; no longer IC20.21
- net N$140: now also IC14.16; no longer IC20.23
- net N$141: now also IC14.9; no longer IC20.13
- net N$143: now also IC14.13; no longer IC20.19
- net N$146: now also IC14.14; no longer IC20.20
- net N$164: now also IC11.11; no longer IC23.15
- net N$165: now also IC11.10; no longer IC23.14
- net N$166: now also IC11.7; no longer IC23.11
- net N$167: now also IC11.8; no longer IC23.12
- net N$168: now also IC11.15; no longer IC23.21
- net N$169: now also IC11.16; no longer IC23.23
- net N$170: now also IC11.9; no longer IC23.13
- net N$172: now also IC11.13; no longer IC23.19
- net N$175: now also IC11.14; no longer IC23.20
- net N$193: now also IC20.11; no longer IC31.15
- net N$194: now also IC20.10; no longer IC31.14
- net N$195: now also IC20.7; no longer IC31.11
- net N$196: now also IC20.8; no longer IC31.12
- net N$197: now also IC20.15; no longer IC31.21
- net N$198: now also IC20.16; no longer IC31.23
- net N$199: now also IC20.9; no longer IC31.13
- net N$201: now also IC20.13; no longer IC31.19
- net N$204: now also IC20.14; no longer IC31.20
- net N$223: now also IC23.11; no longer IC34.15
- net N$224: now also IC23.10; no longer IC34.14
- net N$225: now also IC23.7; no longer IC34.11
- net N$226: now also IC23.8; no longer IC34.12
- net N$227: now also IC23.15; no longer IC34.21
- net N$228: now also IC23.16; no longer IC34.23
- net N$229: now also IC23.9; no longer IC34.13
- net N$231: now also IC23.13; no longer IC34.19
- net N$234: now also IC23.14; no longer IC34.20
- net N$253: now also IC30.11; no longer IC37.15
- net N$254: now also IC30.10; no longer IC37.14
- net N$255: now also IC30.7; no longer IC37.11
- net N$256: now also IC30.8; no longer IC37.12
- net N$262: now also IC30.15; no longer IC37.21
- net N$263: now also IC30.16; no longer IC37.23
- net N$264: now also IC30.9; no longer IC37.13
- net N$266: now also IC30.13; no longer IC37.19
- net N$274: now also IC30.14; no longer IC37.20
- net N$48: now also IC9.11; no longer IC11.15
- net N$49: now also IC9.10; no longer IC11.14
- net N$50: now also IC9.7; no longer IC11.11
- net N$51: now also IC9.8; no longer IC11.12
- net N$52: now also IC9.15; no longer IC11.21
- net N$53: now also IC9.16; no longer IC11.23
- net N$54: now also IC9.9; no longer IC11.13
- net N$56: now also IC9.13; no longer IC11.19
- net N$59: now also IC9.14; no longer IC11.20
- net N$77: now also IC10.11; no longer IC14.15
- net N$78: now also IC10.10; no longer IC14.14
- net N$79: now also IC10.7; no longer IC14.11
- net N$80: now also IC10.8; no longer IC14.12
- net N$81: now also IC10.15; no longer IC14.21
- net N$82: now also IC10.16; no longer IC14.23
- net N$83: now also IC10.9; no longer IC14.13
- net N$85: now also IC10.13; no longer IC14.19
- net N$88: now also IC10.14; no longer IC14.20
- net TCA0_I2C_SCL: now also IC10.4, IC9.4; no longer IC11.7, IC14.7
- net TCA0_I2C_SDA: now also IC10.5, IC9.5; no longer IC11.8, IC14.8
- net TCA1_I2C_SCL: now also IC11.4, IC14.4; no longer IC20.7, IC23.7
- net TCA1_I2C_SDA: now also IC11.5, IC14.5; no longer IC20.8, IC23.8
- net TCA2_I2C_SCL: now also IC17.4, IC20.4; no longer IC17.7, IC31.7
- net TCA2_I2C_SDA: now also IC17.5, IC20.5; no longer IC17.8, IC31.8
- net TCA3_I2C_SCL: now also IC23.4, IC30.4; no longer IC34.7, IC37.7
- net TCA3_I2C_SDA: now also IC23.5, IC30.5; no longer IC34.8, IC37.8
- net VSRC1: now also IC9.1; no longer IC11.24
- net VSRC2: now also IC10.1; no longer IC14.24
- net VSRC3: now also IC11.1; no longer IC23.24
- net VSRC4: now also IC14.1; no longer IC20.24
- net VSRC5: now also IC17.1; no longer IC17.24
- net VSRC6: now also IC20.1; no longer IC31.24
- net VSRC7: now also IC23.1; no longer IC34.24
- net VSRC8: now also IC30.1; no longer IC37.24
Routing:
- net GND: track 1431.4 -> 1561.5 mm, vias 564 -> 504
- net TCA2_I2C_SCL: track 116.9 -> 114.1 mm
- net TCA3_I2C_SCL: track 148.3 -> 145.9 mm
- net N$259: track 10.8 -> 12.2 mm, vias 0 -> 2
- net XO: track 11.7 -> 13.0 mm, vias 0 -> 2
- net TCA1_I2C_SCL: track 89.0 -> 87.7 mm
- net IN1_PORT3: track 9.96 -> 10.9 mm
- net N$110: track 1.10 -> 1.98 mm
- net N$117: track 1.20 -> 2.07 mm
- net N$114: track 12.6 -> 13.5 mm
- net N$83: track 2.63 -> 3.50 mm
- net N$175: track 1.20 -> 2.01 mm
- net N$168: track 1.10 -> 1.91 mm
- net N$172: track 12.6 -> 13.4 mm
- net N$227: track 1.10 -> 1.91 mm
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
Commit message: Update RESET and BOOT part values in hardware design files
Parts:
- BOOT, RESET: value 430182050816 -> 430182043816
Changed lines of the file:
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@@
 <attribute name="VALUE" x="80.735" y="17.135" size="1.27" layer="27" rot="R90"/>
 </element>
-<element name="RESET" library="Wurth_Switch_WS-TASV" library_urn="urn:adsk.eagle:library:18304196" package="430182050816" package3d_urn="urn:adsk.eagle:package:18304299/2" value="430182050816" x="71.01" y="16.38" smashed="yes" rot="R270">
+<element name="RESET" library="Wurth_Switch_WS-TASV" library_urn="urn:adsk.eagle:library:18304196" package="430182050816" package3d_urn="urn:adsk.eagle:package:18304299/2" value="430182043816" x="71.01" y="16.38" smashed="yes" rot="R270">
 <attribute name="DATASHEET-URL" value="https://www.we-online.com/redexpert/spec/430182050816?ae" x="20.21" y="-92.84" size="1.778" layer="27" rot="R270" display="off"/>
 <attribute name="HEIGHT" value="5mm" x="20.21" y="-92.84" size="1.778" layer="27" rot="R270" display="off"/>
@@
 <attribute name="VALUE" x="65.9266" y="19.762" size="1.27" layer="27" rot="R270"/>
 </element>
-<element name="BOOT" library="Wurth_Switch_WS-TASV" library_urn="urn:adsk.eagle:library:18304196" package="430182050816" package3d_urn="urn:adsk.eagle:package:18304299/2" value="430182050816" x="57.4" y="16.35" smashed="yes" rot="R90">
+<element name="BOOT" library="Wurth_Switch_WS-TASV" library_urn="urn:adsk.eagle:library:18304196" package="430182050816" package3d_urn="urn:adsk.eagle:package:18304299/2" value="430182043816" x="57.4" y="16.35" smashed="yes" rot="R90">
 <attribute name="DATASHEET-URL" value="https://www.we-online.com/redexpert/spec/430182050816?ae" x="108.2" y="140.81" size="1.778" layer="27" rot="R90" display="off"/>
 <attribute name="HEIGHT" value="5mm" x="108.2" y="140.81" size="1.778" layer="27" rot="R90" display="off"/>
