File: src/HardwareDesign/Rev0.1.0/PDNode-600 Pro.sch (EAGLE design)
At the start: 652 parts, among them IC1 AP22653W6, IC11 STUSB4710, IC12 TPS552882, IC13 INA219BIDCNT, IC14 STUSB4710, IC15 TPS552882, IC16 INA219BIDCNT, IC17 STUSB4710, IC18 TPS552882, IC19 INA219BIDCNT, IC2 AP22653W6, IC20 STUSB4710, IC21 TPS552882, IC22 INA219BIDCNT, IC23 STUSB4710, IC24 TPS552882, IC25 INA219BIDCNT, IC26 RP2040, IC27 W25Q128JVPIQ, IC28 MCP6001R, IC29 CAT24C512HU5IGT3, IC3 AP22653W6, IC31 STUSB4710, IC32 TPS552882, IC33 INA219BIDCNT, IC34 STUSB4710, IC35 TPS552882, IC36 INA219BIDCNT, IC37 STUSB4710, IC38 TCA9548ARGER, IC39 W5500, IC4 SN74LVC1G04DBVR, IC40 MP2315S, IC41 TPS552882, IC42 MCP23017-E/ML, IC43 MP2315S, IC44 INA219BIDCNT, IC45 MP2315S, IC5 SN74LVC1G04DBVR, IC6 SN74LVC1G04DBVR, IC7 SN74LVC1G04DBVR, IC8 AP22653W6, J1 61400826021, J10 632722100213, J11 632722100213, J2 61400826021, J3 632722100213, J4 632722100213, J5 632722100213, J6 632722100213, J7 632722100213, J8 691244510006, J9 632722100213, T10 IPZ40N04S5L, T11 DMP3013SFV, T12 DMP3013SFV, T13 DMP3013SFV, T14 IPZ40N04S5L, T15 IPZ40N04S5L, T16 DMP3013SFV, T17 DMP3013SFV, T18 DMP3013SFV, T19 IPZ40N04S5L, T20 IPZ40N04S5L, T21 DMP3013SFV, T22 DMP3013SFV, T23 DMP3013SFV, T24 IPZ40N04S5L, T25 IPZ40N04S5L, T26 DMP3013SFV, T27 DMP3013SFV, T28 DMP3013SFV, T29 IPZ40N04S5L, T30 IPZ40N04S5L, T31 DMP3013SFV, T32 DMP3013SFV, T33 DMP3013SFV, T34 IPZ40N04S5L, T35 IPZ40N04S5L, T36 DMP3013SFV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

Commit message: Hardware design update
Parts:
- renumbered J1 to USBA_1-2, J10 to PORT7, J11 to PORT8, J2 to USBA_3-4, J3 to PORT2, J4 to PORT1, J5 to PORT3, J6 to PORT4, J7 to PORT5, J9 to PORT6, S1 to RESET, S2 to BOOT

Commit message: Add BOM
Parts:
- R215, R216, R217: value YC164-JR-0733RL -> 4D03WGJ0332T5E
- T10, T15, T20, T25, T30, T35, T40, T45: value IPZ40N04S5L -> IPZ40N04S5L2R8
- T14, T19, T24, T29, T34, T39, T44, T9: value IPZ40N04S5L -> IPZ40N04S5L-7R4
