File: src/HardwareDesign/1.0.0/SCH_PDCard_101/board_connector.kicad_sch (KiCad schematic)
At the start: 21 parts, among them IC6 TPS74801DRCT, IC7 SN74LVC1G97QDCKRQ1, J2 PCIE EDGE CONNECTOR, U1 24AA02E-OT

Commit message: Baseboard design start
Connections:
- net VBUS_VMON_PORT0: now reaches J2.B10
- net PMIC_VMON_PORT0: now reaches J2.B9
- net PGOOD_COMBIMED renamed PGOOD_COMBINED
- no-connect marks 0 -> 1
Other:
- note added: "Max current: 5.1A per module Pin current capability: 1.1A per Pin (Datasheet) +24V: 8 Pins = 8.8A capability GND: 8 Pins = 8.8A capability"
- note removed: "Max current: 5.1A per module Pin current capability: 1.1A per Pin (Datasheet) +24V: 9 Pins = 9.9A capability GND: 9 Pins = 9.9A capability +24V_SYS: Max 100mA, separate supply for peripherals"
Changed lines of the file:
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@@
 		)
 	)
-	(text "Max current: 5.1A per module\n\nPin current capability: 1.1A per Pin (Datasheet)\n\n+24V: 9 Pins = 9.9A capability\nGND: 9 Pins = 9.9A capability\n\n+24V_SYS: Max 100mA, separate supply for peripherals"
+	(text "Max current: 5.1A per module\n\nPin current capability: 1.1A per Pin (Datasheet)\n\n+24V: 8 Pins = 8.8A capability\nGND: 8 Pins = 8.8A capability"
 		(exclude_from_sim no)
 		(at 138.176 236.474 0)
@@
 		(color 0 0 0 0)
 	)
+	(no_connect
+		(at 114.3 209.55)
+	)
 	(wire
 		(pts
@@
 	(wire
 		(pts
+			(xy 58.42 207.01) (xy 83.82 207.01)
+		)
+		(stroke
+			(width 0)
+			(type default)
+		)
+	)
+	(wire
+		(pts
 			(xy 369.57 86.36) (xy 367.03 86.36)
 		)
@@
 		(pts
 			(xy 121.92 229.87) (xy 121.92 232.41)
+		)
+		(stroke
+			(width 0)
+			(type default)
+		)
+	)
+	(wire
+		(pts
+			(xy 58.42 209.55) (xy 83.82 209.55)
 		)
 		(stroke
@@
 		)
 	)
-	(global_label "PGOOD_COMBIMED"
+	(global_label "PGOOD_COMBINED"
 		(shape input)
 		(at 356.87 73.66 0)
@@
 		)
 		(property "Intersheetrefs" "${INTERSHEET_REFS}"
-			(at 377.0909 73.66 0)
+			(at 376.97 73.66 0)
 			(effects
 				(font
@@
 		)
 	)
-	(global_label "PGOOD_COMBIMED"
+	(global_label "PGOOD_COMBINED"
 		(shape input)
 		(at 58.42 201.93 180)
@@
 		)
 		(property "Intersheetrefs" "${INTERSHEET_REFS}"
-			(at 38.1991 201.93 0)
+			(at 38.32 201.93 0)
 			(effects
 				(font
@@
 		)
 	)
+	(hierarchical_label "VBUS_VMON_PORT0"
+		(shape input)
+		(at 58.42 209.55 180)
+		(effects
+			(font
+				(size 1.27 1.27)
+			)
+			(justify right)
+		)
+	)
 	(hierarchical_label "PD_ENABLE"
 		(shape output)
@@
 		)
 	)
+	(hierarchical_label "PMIC_VMON_PORT0"
+		(shape input)
+		(at 58.42 207.01 180)
+		(effects
+			(font
+				(size 1.27 1.27)
+			)
+			(justify right)
+		)
+	)
