File: src/HardwareDesign/1.0.0/BladeCore-M54_100/BladeCore-M54.kicad_pcb (KiCad board)
At the start: 6 copper layers, 29 x 80.6 mm, 136 parts, among them IC1 RP2354B, IC2 AT24C256C-XHL-T, IC3 W25Q128JVPIQ, IC4 MCP6001RT, IC5 LM4040B30FTA, IC6 W5500, IC7 TPS74801DRCT, IC8 SN74LVC1G97QDCKRQ1, J1 MDT320M03001, J2 Conn_ARM_SWD_TagConnect_TC2030, SW1 B3U-1000P, SW2 B3U-1000P, X1 12MHz 10pF, X2 25MHz 12pF

Commit message: M54 rework
Parts:
- added C57: 100nF 50V, Capacitor_SMD:C_0402_1005Metric, F.Cu at (231.1, 101.5)
- added C59: 1nF 2kV, Capacitor_SMD:C_1206_3216Metric, B.Cu at (223.7, 90.0)
- added D7: SP0503BAHTG, DS_Diode:SOT143, F.Cu at (229.7, 94.3)
- added D8: SS13, Diode_SMD:D_SMA, B.Cu at (223.2, 103.0)
- added IC9: FSUSB42MUX, DS_Peripherals:MSOP-10_3x3mm_P0.5mm, F.Cu at (233.8, 100.3)
- added J3: USB-TYPE-C-018, DS_Connector:USB_C_Receptacle_HCTL_HC-TYPE-C-16P-01A, F.Cu at (230.2, 86.5)
- added R19: 5.1K 1%, Resistor_SMD:R_0402_1005Metric, F.Cu at (232.2, 92.0)
- added R20: 5.1K 1%, Resistor_SMD:R_0402_1005Metric, F.Cu at (234.1, 104.0)
- added R56: 5.1K 1%, Resistor_SMD:R_0402_1005Metric, F.Cu at (227.8, 92.0)
- added R57: 1M 1%, Resistor_SMD:R_1206_3216Metric, F.Cu at (223.8, 89.9)
- D1, R17, R18: moved to B.Cu
- J2: value Conn_ARM_SWD_TagConnect_TC2030 -> SM03B-SRSS-TB; footprint Connector:Tag-Connect_TC2030-IDC-FP_2x03_P1.27mm_Vertical -> DS_Connector:JST_SM03B-SRSS-TB_LF__SN_
- moved J2 53.5 mm to (212.2, 138.9)
- moved R1 8.52 mm to (217.4, 88.3), turned to 0 degrees
- moved C17 7.16 mm to (218.2, 96.2), turned to 90 degrees
- moved IC2 6.17 mm to (222.7, 95.9)
- moved C21 2.30 mm to (222.1, 91.5)
- moved D1 2.12 mm to (219.3, 95.2), turned to 180 degrees
- moved R17 2.11 mm to (219.3, 93.5), turned to 0 degrees
- moved R18 2.09 mm to (219.3, 97.0), turned to 0 degrees
- moved R8 1.99 mm to (222.0, 93.5)
- moved IC5 1.99 mm to (219.6, 91.2)
- moved D4 0.56 mm to (209.2, 145.8)
- moved R51 0.13 mm to (209.1, 151.6), turned to -90 degrees
Connections:
- D5 pad 2: USB_RP_D+ -> USB_D+
- D5 pad 3: USB_RP_D- -> USB_D-
- J1 pad 69: USB_RP_D+ -> USB_D+
- J1 pad 71: USB_RP_D- -> USB_D-
- J2 pad 1: +3.3V -> /Project Architecture/Microcontroller Peripherals/SWDIO
- J2 pad 2: /Project Architecture/Microcontroller Peripherals/SWDIO -> GND
- J2 pad 3: RESET -> /Project Architecture/Microcontroller Peripherals/SWCLK
- R3 pad 2: USB_RP_D- -> /Project Architecture/USB Interface and Power/USB_RP_D-
- R4 pad 1: USB_RP_D+ -> /Project Architecture/USB Interface and Power/USB_RP_D+
- R51 pad 1: VBUS -> VBUS_ISO
- R51 pad 2: VBUS_ISO -> VBUS
Routing:
- net USB_D-: track 0.00 -> 86.3 mm, vias 0 -> 2
- net USB_D+: track 0.00 -> 85.3 mm, vias 0 -> 2
- net VBUS_ONBOARD: track 0.00 -> 48.7 mm, vias 0 -> 11
- net USB_RP_D-: track 47.0 -> 0.00 mm, vias 2 -> 0
- net USB_RP_D+: track 46.9 -> 0.00 mm, vias 2 -> 0
- net /Project Architecture/USB Interface and Power/USB_RP_D-: track 0.00 -> 36.4 mm, vias 0 -> 2
- net /Project Architecture/USB Interface and Power/USB_RP_D+: track 0.00 -> 35.3 mm, vias 0 -> 2
- net USB_ONB_D-: track 0.00 -> 24.4 mm, vias 0 -> 2
- net USB_ONB_D+: track 0.00 -> 23.9 mm, vias 0 -> 2
- net SHIELD: track 0.00 -> 20.8 mm, vias 0 -> 1
- net +5V: track 52.9 -> 73.3 mm, vias 9 -> 11
- net RESET: track 39.6 -> 24.2 mm
- net /Project Architecture/Microcontroller Peripherals/SWCLK: track 35.2 -> 41.3 mm
- net /Project Architecture/Microcontroller Peripherals/I2C0_SCL: track 26.7 -> 20.8 mm
- net /Project Architecture/Microcontroller Peripherals/I2C0_SDA: track 26.8 -> 21.9 mm, vias 2 -> 3
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- added copper zone on In3.Cu, net VBUS_ONBOARD
Other:
- board text removed: "TAGCON"
