File: src/HardwareDesign/1.0.0/BladeCore-M54_100/Block Diagram.kicad_sch (KiCad schematic)
At the start: 0 parts

Commit message: M54 rework
Other:
- note added: "+3.3V"
- note added: "+5V"
- note added: "2280 SIZE M.2 M-KEY CARD"
- note added: "RP2354B"
- note removed: "+??V"
- note removed: "+A3V3"
