File: src/HardwareDesign/1.0.0/BladeCore-M54_100/Power - Sequencing.kicad_sch (KiCad schematic)
At the start: 0 parts

Commit message: M54 rework
Other:
- note added: "+----+------------------------------+-----------+---------------+ | # | Stage | Δt | Total elapsed | +----+------------------------------+-----------+---------------+ | 1 | VIN applied (5.0V) | 0 | 0.000 ms | | 2 | VEN high (TPS74801 EN) | 0 | 0.000 ms | | 3 | VOUT = 3.3V (soft-start) | 4.000 ms | 4.000 ms | | 4 | PGOOD valid | 0 | 4.000 ms | | 5 | RP2354B 3.3V present | 0 | 4.000 ms | | 6 | RP23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"
- note added: ">> RP2354B READY"
