File: src/HardwareDesign/1.0.0/BladeCore-M54_100/Revision History.kicad_sch (KiCad schematic)
At the start: 0 parts

Commit message: M54 rework
Other:
- company: DvidMakesThings -> ${COMPANY}
Changed lines of the file:
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@@
 	(title_block
 		(title "Revision History")
-		(date "2026-02-05")
-		(rev "1.0.0")
-		(company "DvidMakesThings")
+		(date "2026-01-31")
+		(rev "${REVISION}")
+		(company "${COMPANY}")
 	)
-	(text_box "Revision History"
+	(text_box "[${#}] ${TITLE}"
 		(exclude_from_sim no)
 		(at 12.7 15.24 0)
@@
 			(font
 				(face "Times New Roman")
-				(size 6 6)
+				(size 8 8)
 				(thickness 1.2)
 				(bold yes)
-				(color 162 22 34 1)
+				(color 43 49 168 1)
 			)
 		)
@@
 				(width 0)
 				(type solid)
-				(color 162 22 34 1)
+				(color 43 49 168 1)
 			)
 		)
@@
 				(width 0)
 				(type solid)
-				(color 162 22 34 1)
+				(color 43 49 168 1)
 			)
 		)
@@
 						(thickness 0.254)
 						(bold yes)
-						(color 162 22 34 1)
+						(color 43 49 168 1)
 					)
 				)
@@
 						(thickness 0.254)
 						(bold yes)
-						(color 162 22 34 1)
+						(color 43 49 168 1)
 					)
 				)
@@
 						(thickness 0.254)
 						(bold yes)
-						(color 162 22 34 1)
+						(color 43 49 168 1)
 					)
 				)
@@
 						(thickness 0.254)
 						(bold yes)
-						(color 162 22 34 1)
-					)
-				)
-			)
-			(table_cell "07.02.2026"
+						(color 43 49 168 1)
+					)
+				)
+			)
+			(table_cell "31.01.2026"
 				(exclude_from_sim no)
 				(at 134.62 73.66 0)
@@
 					(font
 						(size 1.524 1.524)
-						(color 162 22 34 1)
+						(color 43 49 168 1)
 					)
 					(justify left)
@@
 					(font
 						(size 1.524 1.524)
-						(color 162 22 34 1)
+						(color 43 49 168 1)
 					)
 					(justify left)
@@
 					(font
 						(size 1.524 1.524)
-						(color 162 22 34 1)
+						(color 43 49 168 1)
 					)
 					(justify left)
@@
 					(font
 						(size 1.524 1.524)
-						(color 162 22 34 1)
+						(color 43 49 168 1)
 					)
 					(justify left)
@@
 					(font
 						(size 1.524 1.524)
-						(color 162 22 34 1)
+						(color 43 49 168 1)
 					)
 					(justify left)
@@
 					(font
 						(size 1.524 1.524)
-						(color 162 22 34 1)
+						(color 43 49 168 1)
 					)
 					(justify left)
@@
 					(font
 						(size 1.524 1.524)
-						(color 162 22 34 1)
+						(color 43 49 168 1)
 					)
 					(justify left)
@@
 					(font
 						(size 1.524 1.524)
-						(color 162 22 34 1)
+						(color 43 49 168 1)
 					)
 					(justify left)
@@
 					(font
 						(size 1.524 1.524)
-						(color 162 22 34 1)
+						(color 43 49 168 1)
 					)
 					(justify left)
@@
 					(font
 						(size 1.524 1.524)
-						(color 162 22 34 1)
+						(color 43 49 168 1)
 					)
 					(justify left)
@@
 					(font
 						(size 1.524 1.524)
-						(color 162 22 34 1)
+						(color 43 49 168 1)
 					)
 					(justify left)
@@
 					(font
 						(size 1.524 1.524)
-						(color 162 22 34 1)
+						(color 43 49 168 1)
 					)
 					(justify left)
@@
 					(font
 						(size 1.524 1.524)
-						(color 162 22 34 1)
+						(color 43 49 168 1)
 					)
 					(justify left)
@@
 					(font
 						(size 1.524 1.524)
-						(color 162 22 34 1)
+						(color 43 49 168 1)
 					)
 					(justify left)
@@
 					(font
 						(size 1.524 1.524)
-						(color 162 22 34 1)
+						(color 43 49 168 1)
 					)
 					(justify left)
@@
 					(font
 						(size 1.524 1.524)
-						(color 162 22 34 1)
+						(color 43 49 168 1)
 					)
 					(justify left)
@@
 					(font
 						(size 1.524 1.524)
-						(color 162 22 34 1)
+						(color 43 49 168 1)
 					)
 					(justify left)
@@
 					(font
 						(size 1.524 1.524)
-						(color 162 22 34 1)
+						(color 43 49 168 1)
 					)
 					(justify left)
@@
 					(font
 						(size 1.524 1.524)
-						(color 162 22 34 1)
+						(color 43 49 168 1)
 					)
 					(justify left)
@@
 					(font
 						(size 1.524 1.524)
-						(color 162 22 34 1)
+						(color 43 49 168 1)
 					)
 					(justify left)
@@
 					(font
 						(size 1.524 1.524)
-						(color 162 22 34 1)
+						(color 43 49 168 1)
 					)
 					(justify left)
@@
 					(font
 						(size 1.524 1.524)
-						(color 162 22 34 1)
+						(color 43 49 168 1)
 					)
 					(justify left)
@@
 					(font
 						(size 1.524 1.524)
-						(color 162 22 34 1)
+						(color 43 49 168 1)
 					)
 					(justify left)
@@
 					(font
 						(size 1.524 1.524)
-						(color 162 22 34 1)
+						(color 43 49 168 1)
 					)
 					(justify left)
@@
 					(font
 						(size 1.524 1.524)
-						(color 162 22 34 1)
+						(color 43 49 168 1)
 					)
 					(justify left)
@@
 					(font
 						(size 1.524 1.524)
-						(color 162 22 34 1)
+						(color 43 49 168 1)
 					)
 					(justify left)
@@
 					(font
 						(size 1.524 1.524)
-						(color 162 22 34 1)
+						(color 43 49 168 1)
 					)
 					(justify left)
@@
 					(font
 						(size 1.524 1.524)
-						(color 162 22 34 1)
+						(color 43 49 168 1)
 					)
 					(justify left)
@@
 					(font
 						(size 1.524 1.524)
-						(color 162 22 34 1)
+						(color 43 49 168 1)
 					)
 					(justify left)
@@
 					(font
 						(size 1.524 1.524)
-						(color 162 22 34 1)
+						(color 43 49 168 1)
 					)
 					(justify left)
@@
 					(font
 						(size 1.524 1.524)
-						(color 162 22 34 1)
+						(color 43 49 168 1)
 					)
 					(justify left)
@@
 					(font
 						(size 1.524 1.524)
-						(color 162 22 34 1)
+						(color 43 49 168 1)
 					)
 					(justify left)
@@
 					(font
 						(size 1.524 1.524)
-						(color 162 22 34 1)
+						(color 43 49 168 1)
 					)
 					(justify left)
@@
 					(font
 						(size 1.524 1.524)
-						(color 162 22 34 1)
+						(color 43 49 168 1)
 					)
 					(justify left)
@@
 					(font
 						(size 1.524 1.524)
-						(color 162 22 34 1)
+						(color 43 49 168 1)
 					)
 					(justify left)
@@
 					(font
 						(size 1.524 1.524)
-						(color 162 22 34 1)
-					)
-					(justify left)
+						(color 43 49 168 1)
+					)
+					(justify left)
