File: src/HardwareDesign/1.0.0/BladeCore-M54_100/BladeCore-M54E.kicad_pcb (KiCad board)
At the start: 6 copper layers, 29 x 80.6 mm, 146 parts, among them IC1 RP2354B, IC2 AT24C256C-XHL-T, IC3 W25Q128JVPIQ, IC4 MCP6001RT, IC5 LM4040B30FTA, IC6 W5500, IC7 TPS74801DRCT, IC8 SN74LVC1G97QDCKRQ1, IC9 FSUSB42MUX, J1 MDT320M03001, J2 SM03B-SRSS-TB, J3 USB-TYPE-C-018, SW1 B3U-1000P, SW2 B3U-1000P, X1 12MHz 10pF, X2 25MHz 12pF

Commit message: update readme, add documentation
Changed lines of the file:
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@@
 		(tags "capacitor")
 		(property "Reference" "C34"
-			(at 0.225 4.045 90)
+			(at 2.15 -0.105 90)
 			(layer "F.SilkS")
 			(effects
@@
 		(tags "resistor")
 		(property "Reference" "R46"
-			(at -0.315 4.1 90)
+			(at -1.915 -0.15 90)
 			(layer "F.SilkS")
 			(effects
@@
 		(tags "resistor")
 		(property "Reference" "R44"
-			(at -0.315 4.225 90)
+			(at -1.915 -0.025 90)
 			(layer "F.SilkS")
 			(effects
@@
 		(tags "resistor")
 		(property "Reference" "R42"
-			(at 0.205 4.145 90)
+			(at 2.13 -0.005 90)
 			(layer "F.SilkS")
 			(effects
@@
 		(tags "resistor")
 		(property "Reference" "R39"
-			(at -0.315 4.375 90)
+			(at -1.915 0.125 90)
 			(layer "F.SilkS")
 			(effects
@@
 		(tags "capacitor")
 		(property "Reference" "C33"
-			(at 0.275 4.095 90)
+			(at 2.2 -0.055 90)
 			(layer "F.SilkS")
 			(effects
@@
 		(tags "resistor")
 		(property "Reference" "R41"
-			(at -0.3 4.25 90)
+			(at -1.9 0 90)
 			(layer "F.SilkS")
 			(effects
@@
 		(tags "resistor")
 		(property "Reference" "R40"
-			(at 0.205 4.235 90)
+			(at 2.13 0.085 90)
 			(layer "F.SilkS")
 			(effects

Commit message: finalized 1.0.0 revision, PCB, PCBA ordered
Routing:
- net /Project Architecture/PWR: track 114.1 -> 116.5 mm, vias 6 -> 4
- net GND: track 237.9 -> 237.6 mm, vias 158 -> 163
Other:
- board text added: "HWREV 1.0.0"

Commit message: minor fixes, start with software
Parts:
- removed D2: Green, LED_SMD:LED_0402_1005Metric
- removed JP1: SolderJumper_3_Open, Jumper:SolderJumper-3_P1.3mm_Open_RoundedPad1.0x1.5mm
- removed R62: 1K 1%, Resistor_SMD:R_0402_1005Metric
- added C60: 100nF 50V, Capacitor_SMD:C_0402_1005Metric, B.Cu at (210.1, 140.4)
- added D10: Green, LED_SMD:LED_0402_1005Metric, F.Cu at (208.8, 99.1)
- added D11: Green, LED_SMD:LED_0402_1005Metric, F.Cu at (211.0, 85.9)
- added D9: SS13, Diode_SMD:D_SMA, B.Cu at (209.1, 145.8)
- added IC10: SN74LVC1G97QDCKRQ1, DS_Peripherals:SOT-363_SC-70-6, B.Cu at (210.4, 138.0)
- added R58: 1K 1%, Resistor_SMD:R_0402_1005Metric, F.Cu at (208.8, 101.3)
- added R61: 1K 1%, Resistor_SMD:R_0402_1005Metric, F.Cu at (211.5, 87.6)
- C54: value 1uF 50V -> 4.7uF 25V
- moved D4 0.05 mm to (209.1, 145.8)
Connections:
- net /Project Architecture/Microcontroller/USB_IND renamed Net-(D3-Pad1)
- C52 pad 1: +5V -> REGIN
- C53 pad 1: +5V -> REGIN
- C54 pad 1: /Project Architecture/USB Interface and Power/BIAS -> REGIN
- D4 pad 1: +5V -> REGIN
- D8 pad 1: +5V -> REGIN
- IC1 pad 45: Net-(IC1B-GPIO36) -> HEARTBEAT
- IC7 pad 1: +5V -> REGIN
- IC7 pad 2: +5V -> REGIN
- IC7 pad 4: /Project Architecture/USB Interface and Power/BIAS -> REGIN
- IC7 pad 5: +5V -> REGIN
- J1 pad 10: /Project Architecture/PWR -> +3.3V
- J1 pad 12: /Project Architecture/PWR -> +3.3V
- J1 pad 14: /Project Architecture/PWR -> +5V
- J1 pad 16: /Project Architecture/PWR -> +5V
- R25 pad 1: HEARTBEAT -> unconnected-(R25-R11-Pad1)
- R25 pad 8: Net-(IC1B-GPIO36) -> HEARTBEAT
Routing:
- net /Project Architecture/PWR: track 116.5 -> 0.00 mm, vias 4 -> 0
- net REGIN: track 0.00 -> 75.9 mm, vias 0 -> 12
- net Net-(IC10-Y): track 0.00 -> 55.8 mm, vias 0 -> 3
- net VBUS: track 94.3 -> 40.5 mm, vias 6 -> 5
- net VBUS_ONBOARD: track 48.7 -> 87.8 mm
- net +5V: track 73.3 -> 46.3 mm, vias 11 -> 5
- net +3.3V: track 50.6 -> 68.0 mm, vias 41 -> 44
- net GND: track 237.6 -> 243.9 mm, vias 163 -> 164
- net Net-(IC1B-GPIO36): track 2.53 -> 0.00 mm
- net /Project Architecture/Microcontroller Peripherals/I2C0_SDA: track 21.9 -> 19.8 mm
- net /Project Architecture/Microcontroller Peripherals/I2C0_SCL: track 20.8 -> 18.7 mm
- net /Project Architecture/USB Interface and Power/BIAS: track 1.38 -> 0.00 mm
- net Net-(D11-Pad1): track 0.00 -> 1.22 mm
- net VBUS_ISO: track 2.95 -> 2.43 mm
- added copper zone on B.Cu, net REGIN
- added copper zone on F.Cu, net REGIN
- added copper zone on In3.Cu, net REGIN
- removed copper zone on B.Cu, net +5V
- removed copper zone on F.Cu, net +5V
- removed copper zone on In3.Cu, net +5V
Other:
- board text added: "REG_ON"
- board text removed: "3V3"
- board text removed: "5V"
