File: src/HardwareDesign/1.0.0/BladeCore-M54_100/Project Architecture.kicad_sch (KiCad schematic)
At the start: 3 parts, among them J1 MDT320M03001

Commit message: M54 rework
Parts:
- added R51: 0R 1%, Resistor_SMD:R_1206_3216Metric, symbol DS_Resistor_1206:0R 1% 1206
Connections:
- net VBUS: now also R51.2
- net USB_RP_D+ renamed USB_D+
- net USB_RP_D- renamed USB_D-
- new net VBUS_ISO: R51.1
Other:
- sheet Microcontroller Peripherals ports: added USB_RP_D+, USB_RP_D-; removed none
- sheet USB Interface and Power ports: added USB_RP_D+, USB_RP_D-; removed none
- note added: "Only populate R51 when USB powering is needed"
- company: DvidMakesThings -> ${COMPANY}

Commit message: minor fixes, start with software
Parts:
- removed JP1: SolderJumper_3_Open, Jumper:SolderJumper-3_P1.3mm_Open_RoundedPad1.0x1.5mm, symbol Jumper:SolderJumper_3_Open
- R51: now fitted; now in the parts list
Connections:
- net +3.3V: now also J1.10, J1.12
- net +5V: now also J1.14, J1.16
- removed net PWR: J1.10, J1.12, J1.14, J1.16
Other:
- note removed: "R37 + R38 (5.1 kΩ) + C21 (100 nF): VBUS voltage sense divider and RC filtering for the ADC input; with equal resistors the ADC sees VBUS/2. Only USB-Attached detection"
