File: src/HardwareDesign/1.0.0/BladeCore-M54_100/ethernet_interface.kicad_sch (KiCad schematic)
At the start: 35 parts, among them IC6 W5500, X2 25MHz 12pF

Commit message: M54 rework
Other:
- company: DvidMakesThings -> ${COMPANY}
Changed lines of the file:
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@@
 	(title_block
 		(title "Ethernet Interface")
-		(date "2026-02-05")
-		(rev "1.0.0")
-		(company "DvidMakesThings")
+		(date "2026-01-31")
+		(rev "${REVISION}")
+		(company "${COMPANY}")
 	)
 	(text "DECOUPLING"
@@
 		)
 	)
-	(text_box "Ethernet Interface"
+	(text_box "[${#}] ${TITLE}"
 		(exclude_from_sim no)
 		(at 12.7 16.51 0)
@@
 				(thickness 1.2)
 				(bold yes)
-				(color 162 22 34 1)
+				(color 43 49 168 1)
 			)
 		)
