File: src/HardwareDesign/1.0.0/BladeCore-M54_100/microcontroller.kicad_sch (KiCad schematic)
At the start: 32 parts, among them IC1 RP2354B

Commit message: M54 rework
Other:
- company: DvidMakesThings -> ${COMPANY}
Changed lines of the file:
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@@
 	(title_block
 		(title "Microcontroller")
-		(date "2026-02-05")
-		(rev "1.0.0")
-		(company "DvidMakesThings")
+		(date "2026-01-31")
+		(rev "${REVISION}")
+		(company "${COMPANY}")
 	)
 	(text "I2C PULLUP"
@@
 		)
 	)
-	(text_box "Microcontroller"
+	(text_box "[${#}] ${TITLE}"
 		(exclude_from_sim no)
 		(at 12.7 19.05 0)
@@
 				(thickness 1.2)
 				(bold yes)
-				(color 162 22 34 1)
+				(color 43 49 168 1)
 			)
 		)

Commit message: minor fixes, start with software
Connections:
- net HEARTBEAT: now also IC1.45 (GPIO36), R25.8 (R12); no longer R25.1 (R11)
- net USB_IND: no longer names the net of D3.1, R34.2
- no-connect marks 0 -> 1
