File: src/HardwareDesign/1.0.0/BladeCore-M54_100/microcontroller_peripherals.kicad_sch (KiCad schematic)
At the start: 45 parts, among them IC1 RP2354B, IC2 AT24C256C-XHL-T, IC3 W25Q128JVPIQ, IC4 MCP6001RT, IC5 LM4040B30FTA, J2 Conn_ARM_SWD_TagConnect_TC2030, SW1 B3U-1000P, SW2 B3U-1000P, X1 12MHz 10pF

Commit message: M54 rework
Parts:
- removed J2: Conn_ARM_SWD_TagConnect_TC2030, Connector:Tag-Connect_TC2030-IDC-FP_2x03_P1.27mm_Vertical, symbol Connector:Conn_ARM_SWD_TagConnect_TC2030
- added J2: SM03B-SRSS-TB, DS_Connector:JST_SM03B-SRSS-TB_LF__SN_, symbol DS_Connector:DebugProbe SWD
Connections:
- net GND: now also J2.2 (GND), J2.S1 (SHIELD), J2.S2 (SHIELD)
- net SWCLK: now also J2.3 (SWDAT)
- net SWDIO: now also J2.1 (SWCLK)
- no-connect marks 1 -> 0
Other:
- company: DvidMakesThings -> ${COMPANY}
