File: src/HardwareDesign/1.0.0/PDCard-4242_100/PDNode-PDCard-4242.kicad_pcb (KiCad board)
At the start: 6 copper layers, 53.9 x 29.9 mm, 75 parts, among them IC1 MCP1702T-3302E/CB, IC2 MPQ4242GVE-0001-AEC1-P, IC20 24AA02E-OT, IC3 INA219BIDCNT, IC5 SN74LVC1G97QDCKRQ1, J1 USB-TYPE-C-018, J2 PCIE EDGE CONNECTOR, T1 DMN4008LFG-7

Commit message: hardware design is close to final status
Routing:
- net GND: track 98.4 -> 98.6 mm, vias 95 -> 101
- net /Project Architecture/USB-PD Source Controller/I2C_SDA: vias 4 -> 5
Changed lines of the file:
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@@
 		)
 		(embedded_fonts no)
+		(model "${KICAD_LIB_GITHUB}/DS_Peripherals/3D/MPQ4242GVE.STEP"
+			(offset
+				(xyz -2 -2.5 0.01)
+			)
+			(scale
+				(xyz 1 1 1)
+			)
+			(rotate
+				(xyz -0 -0 -0)
+			)
+		)
 	)
 	(footprint "DS_Capacitor:C_0402_1005Metric"
@@
 			(at 0 1.17 270)
 			(layer "B.SilkS")
+			(hide yes)
 			(effects
 				(font
@@
 	)
 	(via
+		(at 205.375 153.675)
+		(size 0.4)
+		(drill 0.2)
+		(layers "F.Cu" "B.Cu")
+		(net 2)
+	)
+	(via
 		(at 220.875 150.725)
 		(size 0.4)
@@
 	)
 	(via
-		(at 206.075 149.625)
+		(at 205.575 149.625)
 		(size 0.4)
 		(drill 0.2)
@@
 	)
 	(via
+		(at 231.075 148.325)
+		(size 0.4)
+		(drill 0.2)
+		(layers "F.Cu" "B.Cu")
+		(net 2)
+	)
+	(via
 		(at 222.075 150.725)
 		(size 0.4)
@@
 	)
 	(via
+		(at 205.275 146.825)
+		(size 0.4)
+		(drill 0.2)
+		(layers "F.Cu" "B.Cu")
+		(net 2)
+	)
+	(via
 		(at 227.246455 157.223131)
 		(size 0.4)
@@
 	)
 	(via
+		(at 208.375 149.925)
+		(size 0.4)
+		(drill 0.2)
+		(layers "F.Cu" "B.Cu")
+		(net 2)
+	)
+	(via
 		(at 209.375 142.825)
 		(size 0.4)
@@
 	)
 	(via
+		(at 205.275 148.025)
+		(size 0.4)
+		(drill 0.2)
+		(layers "F.Cu" "B.Cu")
+		(net 2)
+	)
+	(via
 		(at 194.375 155.425)
 		(size 0.4)
@@
 	)
 	(via
+		(at 229.575 141.525)
+		(size 0.4)
+		(drill 0.2)
+		(layers "F.Cu" "B.Cu")
+		(net 2)
+	)
+	(via
 		(at 225.246455 155.873131)
 		(size 0.4)
@@
 	)
 	(segment
+		(start 206.075 148.985)
+		(end 206.075 149.125)
+		(width 0.174)
+		(layer "B.Cu")
+		(net 2)
+	)
+	(segment
 		(start 227.25 155.876676)
 		(end 227.246455 155.873131)
@@
 	)
 	(segment
+		(start 206.075 149.125)
+		(end 205.575 149.625)
+		(width 0.174)
+		(layer "B.Cu")
+		(net 2)
+	)
+	(segment
 		(start 227.25 160.175)
 		(end 227.25 157.475)
@@
 	)
 	(segment
-		(start 206.075 148.985)
-		(end 206.075 149.625)
-		(width 0.174)
-		(layer "B.Cu")
-		(net 2)
-	)
-	(segment
 		(start 211.25 157.025)
 		(end 211.25 160.175)
@@
 	)
 	(segment
-		(start 207.275 149.675)
-		(end 205.625 151.325)
+		(start 205.875 152.225)
+		(end 206.275 152.625)
 		(width 0.2)
 		(layer "F.Cu")
@@
 	)
 	(segment
-		(start 207.275 148.925)
-		(end 207.275 149.675)
+		(start 207.965 148.525)
+		(end 207.675 148.525)
 		(width 0.2)
 		(layer "F.Cu")
@@
 	)
 	(segment
-		(start 222.99 146.535)
-		(end 222.77 146.755)
-		(width 0.174)
+		(start 208.265 148.825)
+		(end 207.965 148.525)
+		(width 0.2)
 		(layer "F.Cu")
 		(net 3)
 	)
 	(segment
-		(start 222.77 146.755)
-		(end 222.05 146.755)
-		(width 0.174)
+		(start 207.275 148.925)
+		(end 207.275 149.425)
+		(width 0.2)
 		(layer "F.Cu")
 		(net 3)
 	)
 	(segment
-		(start 205.625 152.425)
-		(end 205.825 152.625)
+		(start 207.675 148.525)
+		(end 207.275 148.925)
 		(width 0.2)
 		(layer "F.Cu")
@@
 	)
 	(segment
-		(start 205.825 152.625)
-		(end 207.9125 152.625)
-		(width 0.2)
+		(start 222.99 146.535)
+		(end 222.77 146.755)
+		(width 0.174)
 		(layer "F.Cu")
 		(net 3)
 	)
 	(segment
-		(start 220.785 148.02)
+		(start 222.77 146.755)
 		(end 222.05 146.755)
 		(width 0.174)
@@
 	)
 	(segment
-		(start 207.9125 152.625)
-		(end 207.575 152.625)
-		(width 0.2)
+		(start 220.785 148.02)
+		(end 222.05 146.755)
+		(width 0.174)
 		(layer "F.Cu")
 		(net 3)
 	)
 	(segment
-		(start 218.3625 148.02)
-		(end 220.4625 148.02)
-		(width 0.174)
+		(start 206.275 152.625)
+		(end 207.9125 152.625)
+		(width 0.2)
 		(layer "F.Cu")
 		(net 3)
 	)
 	(segment
-		(start 207.675 148.525)
-		(end 207.275 148.925)
+		(start 207.9125 152.625)
+		(end 207.575 152.625)
 		(width 0.2)
 		(layer "F.Cu")
@@
 	)
 	(segment
-		(start 208.265 148.825)
-		(end 207.965 148.525)
+		(start 207.275 149.425)
+		(end 205.875 150.825)
 		(width 0.2)
 		(layer "F.Cu")
@@
 	)
 	(segment
-		(start 207.965 148.525)
-		(end 207.675 148.525)
+		(start 205.875 150.825)
+		(end 205.875 152.225)
 		(width 0.2)
 		(layer "F.Cu")
@@
 	)
 	(segment
-		(start 224.35 146.535)
-		(end 222.99 146.535)
+		(start 218.3625 148.02)
+		(end 220.4625 148.02)
 		(width 0.174)
 		(layer "F.Cu")
@@
 	)
 	(segment
-		(start 205.625 151.325)
-		(end 205.625 152.425)
-		(width 0.2)
+		(start 224.35 146.535)
+		(end 222.99 146.535)
+		(width 0.174)
 		(layer "F.Cu")
 		(net 3)
@@
 		(net 14)
 	)
+	(via
+		(at 209.275 141.825)
+		(size 0.4)
+		(drill 0.2)
+		(layers "F.Cu" "B.Cu")
+		(net 14)
+	)
 	(segment
 		(start 213.075 154.225)
@@
 	)
 	(segment
-		(start 202.323606 152.625)
-		(end 205.075 152.625)
+		(start 201.9875 153.7625)
+		(end 201.9875 152.625)
 		(width 0.2)
 		(layer "F.Cu")
@@
 	)
 	(segment
-		(start 201.9875 153.7625)
-		(end 201.9875 152.625)
+		(start 206.875 148.775)
+		(end 207.525 148.125)
+		(width 0.2)
+		(layer "F.Cu")
+		(net 23)
+	)
+	(segment
+		(start 205.475 152.225)
+		(end 205.475 150.75)
 		(width 0.2)
 		(layer "F.Cu")
@@
 	)
 	(segment
+		(start 207.525 148.125)
+		(end 207.975 148.125)
+		(width 0.2)
+		(layer "F.Cu")
+		(net 23)
+	)
+	(segment
 		(start 195.975 145.025)
 		(end 195.775 145.025)
@@
 	)
 	(segment
-		(start 197.175 145.025)
-		(end 197.177027 145.022973)
-		(width 0.4)
+		(start 205.075 152.625)
+		(end 205.475 152.225)
+		(width 0.2)
 		(layer "F.Cu")
 		(net 23)
 	)
 	(segment
-		(start 205.275 152.425)
-		(end 205.275 151.175)
-		(width 0.2)
+		(start 197.175 145.025)
+		(end 197.177027 145.022973)
+		(width 0.4)
 		(layer "F.Cu")
 		(net 23)
@@
 	)
 	(segment
+		(start 205.475 150.75)
+		(end 206.875 149.35)
+		(width 0.2)
+		(layer "F.Cu")
+		(net 23)
+	)
+	(segment
 		(start 195.977027 145.022973)
 		(end 195.975 145.025)
@@
 	)
 	(segment
-		(start 206.875 148.775)
-		(end 207.525 148.125)
-		(width 0.2)
-		(layer "F.Cu")
-		(net 23)
-	)
-	(segment
 		(start 199.725 145.025)
 		(end 201.975 145.025)
@@
 	)
 	(segment
-		(start 202.321957 152.626649)
-		(end 202.323606 152.625)
+		(start 206.875 149.35)
+		(end 206.875 148.775)
 		(width 0.2)
 		(layer "F.Cu")
@@
 	)
 	(segment
-		(start 205.075 152.625)
-		(end 205.275 152.425)
-		(width 0.2)
-		(layer "F.Cu")
-		(net 23)
-	)
-	(segment
 		(start 198.475 149.639)
 		(end 198.865008 149.639)
@@
 	)
 	(segment
-		(start 207.525 148.125)
-		(end 207.975 148.125)
-		(width 0.2)
-		(layer "F.Cu")
-		(net 23)
-	)
-	(segment
 		(start 198.865008 145.211)
 		(end 199.051008 145.025)
@@
 	)
 	(segment
-		(start 205.275 151.175)
-		(end 206.875 149.575)
-		(width 0.2)
-		(layer "F.Cu")
-		(net 23)
-	)
-	(segment
 		(start 197.177027 145.022973)
 		(end 197.663281 145.022973)
@@
 	)
 	(segment
-		(start 206.875 149.575)
-		(end 206.875 148.775)
-		(width 0.2)
-		(layer "F.Cu")
-		(net 23)
-	)
-	(segment
 		(start 199.053035 149.827027)
 		(end 199.386719 149.827027)
@@
 	)
 	(segment
+		(start 207.975 148.125)
+		(end 208.275 147.825)
+		(width 0.2)
+		(layer "F.Cu")
+		(net 23)
+	)
+	(segment
 		(start 201.375 155.315)
 		(end 201.375 154.375)
@@
 	)
 	(segment
-		(start 207.975 148.125)
-		(end 208.275 147.825)
+		(start 202.323606 152.625)
+		(end 205.075 152.625)
 		(width 0.2)
 		(layer "F.Cu")
@@
 		(layer "F.Cu")
 		(net 23)
+	)
+	(segment
+		(start 202.321957 152.626649)
+		(end 202.323606 152.625)
+		(width 0.2)
+		(layer "F.Cu")
+		(net 23)
