File: src/HardwareDesign/1.0.0/PDCard-4242_100/Block Diagram.kicad_sch (KiCad schematic)
At the start: 0 parts

Commit message: update readme, add documentation
Other:
- note added: "USB-C"
Changed lines of the file:
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@@
+	(text "INTEGRATED\nBUCK-BOOST"
+		(exclude_from_sim no)
+		(at 213.36 91.948 0)
+		(effects
+			(font
+				(size 2.54 2.54)
+				(thickness 0.508)
+				(bold yes)
+				(color 0 0 0 1)
+			)
+		)
+	)
 	(text "INTEGRATED\nBUCK-BOOST"
 		(exclude_from_sim no)
@@
 		(effects
 			(font
+				(size 2.54 2.54)
+				(thickness 0.508)
+				(bold yes)
+				(color 0 0 0 1)
+			)
+		)
+	)
+	(text "USB-C"
+		(exclude_from_sim no)
+		(at 289.56 133.35 0)
+		(effects
+			(font
