File: src/HardwareDesign/1.0.0/PDCard-4242_100/usb_pd_source_controller.kicad_sch (KiCad schematic)
At the start: 55 parts, among them IC2 MPQ4242GVE-0001-AEC1-P, IC3 INA219BIDCNT, T1 DMN4008LFG-7

Commit message: update readme, add documentation
Parts:
- renumbered PDAT1 to PDA1, PDEN1 to PDE1, PDOUT1 to PDO1, VMON1 to TP1, V24F1 to VF24

Commit message: finalized 1.0.0 revision, PCB, PCBA ordered
Parts:
- R17, R18: LCSC_PART C25101 -> C2909330
Changed lines of the file:
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@@
 			)
 		)
-		(property "Datasheet" ""
+		(property "Datasheet" "https://jlcpcb.com/api/file/downloadByFileSystemAccessId/8590208205541711872"
 			(at 280.416 168.148 0)
 			(show_name yes)
@@
 			)
 		)
-		(property "LCSC_PART" "C25101"
+		(property "LCSC_PART" "C2909330"
 			(at 278.384 168.148 0)
 			(show_name yes)
@@
 			)
 		)
-		(property "Datasheet" ""
+		(property "Datasheet" "https://jlcpcb.com/api/file/downloadByFileSystemAccessId/8590208205541711872"
 			(at 280.416 178.308 0)
 			(show_name yes)
@@
 			)
 		)
-		(property "LCSC_PART" "C25101"
+		(property "LCSC_PART" "C2909330"
 			(at 278.384 178.308 0)
 			(show_name yes)

Commit message: minor fixes, start with software
Parts:
- C1, C10: LCSC_PART C696814 -> C215892; MFR KEMET -> Vishay; MPN T521D107M025ATE040 -> T55D107M025C0060
- C36, C37: LCSC_PART C107050 -> C20069334; MFR YAGEO -> HRE; MPN CC0603JRNPO9BN391 -> CGA0402C0G391J500GT
Changed lines of the file:
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@@
 			)
 		)
-		(property "Datasheet" "https://content.kemet.com/datasheets/kem_t2076_t52x-530.pdf"
+		(property "Datasheet" "https://jlcpcb.com/api/file/downloadByFileSystemAccessId/8590224151765426176"
 			(at 311.15 143.256 0)
 			(show_name yes)
@@
 			)
 		)
-		(property "LCSC_PART" "C696814"
+		(property "LCSC_PART" "C215892"
 			(at 311.15 139.192 0)
 			(show_name yes)
@@
 			)
 		)
-		(property "MPN" "T521D107M025ATE040"
+		(property "MPN" "T55D107M025C0060"
 			(at 311.15 135.128 0)
 			(show_name yes)
@@
 			)
 		)
-		(property "MFR" "KEMET"
+		(property "MFR" "Vishay "
 			(at 311.15 147.574 0)
 			(show_name yes)
@@
 			)
 		)
-		(property "Datasheet" "https://jlcpcb.com/api/file/downloadByFileSystemAccessId/8588898749053063168"
+		(property "Datasheet" "https://jlcpcb.com/api/file/downloadByFileSystemAccessId/8590919194240503808"
 			(at 279.4 201.168 0)
 			(show_name yes)
@@
 			)
 		)
-		(property "Description" "390pF 50V NP0 ±5% 0603 Multilayer Ceramic Capacitors MLCC - SMD/SMT ROHS"
+		(property "Description" "390pF 50V C0G ±5% 0402 Multilayer Ceramic Capacitors MLCC - SMD/SMT ROHS"
 			(at 279.4 205.232 0)
 			(show_name yes)
@@
 			)
 		)
-		(property "LCSC_PART" "C107050"
+		(property "LCSC_PART" "C20069334"
 			(at 279.4 199.136 0)
 			(show_name yes)
@@
 			)
 		)
-		(property "MFR" "YAGEO"
+		(property "MFR" "HRE"
 			(at 279.4 203.2 0)
 			(show_name yes)
@@
 			)
 		)
-		(property "MPN" "CC0603JRNPO9BN391"
+		(property "MPN" "CGA0402C0G391J500GT"
 			(at 279.4 209.296 0)
 			(show_name yes)
@@
 			)
 		)
-		(property "Datasheet" "https://jlcpcb.com/api/file/downloadByFileSystemAccessId/8588898749053063168"
+		(property "Datasheet" "https://jlcpcb.com/api/file/downloadByFileSystemAccessId/8590919194240503808"
 			(at 297.18 201.168 0)
 			(show_name yes)
@@
 			)
 		)
-		(property "Description" "390pF 50V NP0 ±5% 0603 Multilayer Ceramic Capacitors MLCC - SMD/SMT ROHS"
+		(property "Description" "390pF 50V C0G ±5% 0402 Multilayer Ceramic Capacitors MLCC - SMD/SMT ROHS"
 			(at 297.18 205.232 0)
 			(show_name yes)
@@
 			)
 		)
-		(property "LCSC_PART" "C107050"
+		(property "LCSC_PART" "C20069334"
 			(at 297.18 199.136 0)
 			(show_name yes)
@@
 			)
 		)
-		(property "MFR" "YAGEO"
+		(property "MFR" "HRE"
 			(at 297.18 203.2 0)
 			(show_name yes)
@@
 			)
 		)
-		(property "MPN" "CC0603JRNPO9BN391"
+		(property "MPN" "CGA0402C0G391J500GT"
 			(at 297.18 209.296 0)
 			(show_name yes)
@@
 			)
 		)
-		(property "Datasheet" "https://content.kemet.com/datasheets/kem_t2076_t52x-530.pdf"
+		(property "Datasheet" "https://jlcpcb.com/api/file/downloadByFileSystemAccessId/8590224151765426176"
 			(at 33.02 145.796 0)
 			(show_name yes)
@@
 			)
 		)
-		(property "LCSC_PART" "C696814"
+		(property "LCSC_PART" "C215892"
 			(at 33.02 141.732 0)
 			(show_name yes)
@@
 			)
 		)
-		(property "MPN" "T521D107M025ATE040"
+		(property "MPN" "T55D107M025C0060"
 			(at 33.02 137.668 0)
 			(show_name yes)
@@
 			)
 		)
-		(property "MFR" "KEMET"
+		(property "MFR" "Vishay "
 			(at 33.02 150.114 0)
 			(show_name yes)
