File: src/HardwareDesign/1.0.0/PDNode-600_Pro_Baseboard_100/Power - Sequencing.kicad_sch (KiCad schematic)
At the start: 0 parts

Commit message: baseboard development
Changed lines of the file:
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@@
 			(font
 				(face "Times New Roman")
-				(size 6 6)
+				(size 8 8)
 				(thickness 1.2)
 				(bold yes)

Commit message: hardware design is close to final status
Other:
- note removed: ">> NORMAL >> OPERATION"
- note removed: "Time [ms]"
- note removed: "Voltage [V]"
