File: src/HardwareDesign/1.0.0/PDNode-600_Pro_Baseboard_100/Project Architecture.kicad_sch (KiCad schematic)
At the start: 3 parts, among them J1 HR911105A

Commit message: M54 rework
Other:
- company: DvidMakesThings -> ${COMPANY}
Changed lines of the file:
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@@
 	(title_block
 		(title "Project Architecture")
-		(date "2026-02-05")
-		(rev "1.0.0")
-		(company "DvidMakesThings")
+		(date "2025-01-12")
+		(rev "${REVISION}")
+		(company "${COMPANY}")
 	)
 	(arc

Commit message: baseboard development
Other:
- sheet USB Interface renamed USB Interface and Display
- sheet External Power Connectors ports: added ADC_24V; removed none
- moved on the sheet: C1, R1

Commit message: finalized 1.0.0 revision, PCB, PCBA ordered
Parts:
- removed J1: HR911105A, DS_Connector:100BASE_MAGJACK, symbol DS_Connector:HR911105A
- added J1: J1B1211CCD, DS_Connector:J1B1211CCD, symbol DS_Connector:J1B1211CCD
- C1: footprint Capacitor_SMD:C_1206_3216Metric -> DS_Capacitor:C_1206_3216Metric
- R1: footprint Resistor_SMD:R_1206_3216Metric -> DS_Resistor:R_1206_3216Metric
Connections:
- net +3.3V: now also J1.10 (GREEN+), J1.12 (YELLOW+)
- net BladeCore-M54/ACTLED: now also J1.9 (GREEN-)
- net BladeCore-M54/LINKLED: now also J1.11 (YELLOW-)
- net BladeCore-M54/RCT: now also J1.5 (P5/RCT)
- net BladeCore-M54/RD+: now also J1.4 (RD+)
- net BladeCore-M54/RD-: now also J1.6 (RD-)
- net BladeCore-M54/TCT: now also J1.2 (P4/TCT)
- net BladeCore-M54/TD+: now also J1.1 (TD+)
- net BladeCore-M54/TD-: now also J1.3 (TD-)
- net GND: now also J1.8 (GND)
- net SHIELD: now also J1.13 (SHIELD), J1.14 (SHIELD)
- no-connect marks 3 -> 1
Other:
- sheet BladeCore-M54 ports: added SPI_CS; removed none
- sheet USB Interface and Display ports: added I2C1_SCL, I2C1_SDA, SPI_CLK, SPI_CS, SPI_MISO, SPI_MOSI; removed USB_DBG_D+, USB_DBG_D-
