File: src/HardwareDesign/1.0.0/PDNode-600_Pro_Baseboard_100/TCA9548_port_controller.kicad_sch (KiCad schematic)
At the start: 13 parts, among them IC4 TCA9548ARGER

Commit message: M54 rework
Other:
- company: DvidMakesThings -> ${COMPANY}
Changed lines of the file:
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@@
 	(title_block
 		(title "TCA9548 Port Controller")
-		(date "2026-02-05")
-		(rev "1.0.0")
-		(company "DvidMakesThings")
+		(date "2025-01-12")
+		(rev "${REVISION}")
+		(company "${COMPANY}")
 	)
 	(text "TCA9548 1-TO-8 I2C MULTIPLEXER"

Commit message: finalized 1.0.0 revision, PCB, PCBA ordered
Parts:
- C64: footprint Capacitor_SMD:C_0402_1005Metric -> DS_Capacitor:C_0402_1005Metric
- R25, R26, R27, R28, R42, R43, R46, R47: footprint Resistor_SMD:R_Array_Convex_4x0603 -> DS_Resistor:R_Array_Convex_4x0603
- R41, R44, R45: footprint Resistor_SMD:R_0402_1005Metric -> DS_Resistor:R_0402_1005Metric
Changed lines of the file:
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@@
 	)
 	(junction
-		(at 236.22 95.25)
-		(diameter 0)
-		(color 0 0 0 0)
-	)
-	(junction
 		(at 189.23 95.25)
 		(diameter 0)
@@
 	(wire
 		(pts
-			(xy 236.22 95.25) (xy 290.83 95.25)
-		)
-		(stroke
-			(width 0)
-			(type default)
-		)
-	)
-	(wire
-		(pts
 			(xy 127 160.02) (xy 138.43 160.02)
 		)
@@
 			)
 		)
-		(property "Footprint" "Resistor_SMD:R_0402_1005Metric"
+		(property "Footprint" "DS_Resistor:R_0402_1005Metric"
 			(at 70.104 133.858 0)
 			(effects
@@
 			)
 		)
-		(property "Footprint" "Resistor_SMD:R_Array_Convex_4x0603"
+		(property "Footprint" "DS_Resistor:R_Array_Convex_4x0603"
 			(at 201.93 107.95 0)
 			(show_name yes)
@@
 			)
 		)
-		(property "Footprint" "Resistor_SMD:R_Array_Convex_4x0603"
+		(property "Footprint" "DS_Resistor:R_Array_Convex_4x0603"
 			(at 137.16 124.46 0)
 			(show_name yes)
@@
 			)
 		)
-		(property "Footprint" "Resistor_SMD:R_Array_Convex_4x0603"
+		(property "Footprint" "DS_Resistor:R_Array_Convex_4x0603"
 			(at 147.32 139.7 0)
 			(show_name yes)
@@
 			)
 		)
-		(property "Footprint" "Resistor_SMD:R_0402_1005Metric"
+		(property "Footprint" "DS_Resistor:R_0402_1005Metric"
 			(at 61.976 136.398 0)
 			(effects
@@
 			)
 		)
-		(property "Footprint" "Resistor_SMD:R_Array_Convex_4x0603"
+		(property "Footprint" "DS_Resistor:R_Array_Convex_4x0603"
 			(at 154.94 107.95 0)
 			(show_name yes)
@@
 			)
 		)
-		(property "Footprint" "Capacitor_SMD:C_0402_1005Metric"
+		(property "Footprint" "DS_Capacitor:C_0402_1005Metric"
 			(at 29.21 142.494 0)
 			(show_name yes)
@@
 			)
 		)
-		(property "Footprint" "Resistor_SMD:R_Array_Convex_4x0603"
+		(property "Footprint" "DS_Resistor:R_Array_Convex_4x0603"
 			(at 179.07 107.95 0)
 			(show_name yes)
@@
 			)
 		)
-		(property "Footprint" "Resistor_SMD:R_Array_Convex_4x0603"
+		(property "Footprint" "DS_Resistor:R_Array_Convex_4x0603"
 			(at 147.32 170.18 0)
 			(show_name yes)
@@
 			)
 		)
-		(property "Footprint" "Resistor_SMD:R_Array_Convex_4x0603"
+		(property "Footprint" "DS_Resistor:R_Array_Convex_4x0603"
 			(at 226.06 107.95 0)
 			(show_name yes)
@@
 			)
 		)
-		(property "Footprint" "Resistor_SMD:R_Array_Convex_4x0603"
+		(property "Footprint" "DS_Resistor:R_Array_Convex_4x0603"
 			(at 137.16 154.94 0)
 			(show_name yes)
@@
 			)
 		)
-		(property "Footprint" "Resistor_SMD:R_0402_1005Metric"
+		(property "Footprint" "DS_Resistor:R_0402_1005Metric"
 			(at 77.978 109.474 0)
 			(effects

Commit message: minor fixes, start with software
Parts:
- R41: now fitted; now in the parts list
