File: src/HardwareDesign/1.0.0/PDNode-600_Pro_Baseboard_100/bladecore-m54.kicad_sch (KiCad schematic)
At the start: 5 parts, among them IC2 CD74HC4067QRGYRQ1, J2 MDT320M03001

Commit message: M54 rework
Other:
- company: DvidMakesThings -> ${COMPANY}
Changed lines of the file:
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@@
 	(title_block
 		(title "Microcontroller")
-		(date "2026-02-05")
-		(rev "1.0.0")
-		(company "DvidMakesThings")
+		(date "2025-01-12")
+		(rev "${REVISION}")
+		(company "${COMPANY}")
 	)
 	(text "CD74HC4067QRGYRQ1:\n==============\n- Ron 160 Ω max: compared to THE divider (90.9K/10K) Thevenin (~9 kΩ), \n   that's a ~1-2% scale error worst case if the ADC input were purely \n   resistive. With 1 nF at the ADC INPUT, the mux mostly just charges \n   that cap, so the practical impact is smaller.\n- Leakage 800 nA max: into ~9 kΩ source is only ~7 mV worst-case \n   equivalent error.\n- Off capacitances (5 pF / 50 pF): 100R + 1 nF kills that nicely. \n   Dummy conversion (throwaway sample) after switching helps too.\n   R = 9K + 100R = 9.1K\n   C = 1nF\n   t = 9.1 us\n   -> 5t = 45us after switching the MUX channel is settled\n"

Commit message: baseboard development
Parts:
- removed J2: MDT320M03001, DS_Connector:BladeCore-M54, symbol DS_Connector:BladeCore-M54
- added J2: MDT580M01001, DS_Connector:BladeCore-M54E-5.8mm, symbol DS_Connector:BladeCore-M54E
- added ST1: M2.5, DS_Test:Round Standoff Threaded M2.5 Steel, symbol DS_Test:PCIe Hole M2.5 4.5mm
Connections:
- net +3.3V: now also J2.10 (PWR), J2.12 (PWR), J2.14 (PWR), J2.16 (PWR)
- net 5V_BUCK_EN: now also J2.21 (GPIO16)
- net ACTLED: now also J2.18 (LINKLED)
- net ADC_24V: now also J2.46 (ADC0)
- net ADC_3V3A: now also J2.54 (ADC4)
- net ADC_3V3SW: now also J2.52 (ADC3)
- net ADC_5VA: now also J2.50 (ADC2)
- net ADC_5VSW: now also J2.48 (ADC1)
- net GND: now also J2.1 (GND), J2.11 (GND), J2.2 (GND), J2.22 (GND), J2.23 (GND), J2.26 (GND), J2.32 (GND), J2.38 (GND), J2.41 (GND), J2.42 (GND), J2.44 (GND), J2.58 (GND), J2.67 (GND), J2.68 (GND), J2.70 (GND), J2.73 (GND), J2.SH1 (SHIELD), ST1.1
- net I2C1_SCL: now also J2.51 (GPIO3)
- net I2C1_SDA: now also J2.53 (GPIO2)
- net LINKLED: now also J2.20 (ACTLED)
- net MCP_RESET: now also J2.8 (GPIO25)
- net MUX_OUT: now also J2.56 (ADC5)
- net MUX_S0: now also J2.3 (GPIO24)
- net MUX_S1: now also J2.5 (GPIO23)
- net MUX_S2: now also J2.7 (GPIO22)
- net MUX_S3: now also J2.9 (GPIO21)
- net PAC_ALERT_P01: now also J2.13 (GPIO20)
- net PAC_ALERT_P23: now also J2.15 (GPIO19)
- net PD_IRQ_EVENT_A: now also J2.6 (GPIO26)
- net PD_IRQ_EVENT_A2: now also J2.57 (GPIO0)
- net PD_IRQ_EVENT_B: now also J2.4 (GPIO27)
- net PD_IRQ_EVENT_B2: now also J2.55 (GPIO1)
- net PGOOD_SYSPMIC: now also J2.19 (GPIO17)
- net RCT: now also J2.24 (RCT)
- net RD+: now also J2.28 (ETH_RD+)
- net RD-: now also J2.30 (ETH_RD-)
- net SPI_CLK: now also J2.45 (GPIO6)
- net SPI_CS_PORT0: now also J2.25 (GPIO15)
- net SPI_CS_PORT1: now also J2.27 (GPIO14)
- net SPI_CS_PORT2: now also J2.29 (GPIO13)
- net SPI_CS_PORT3: now also J2.31 (GPIO12)
- net SPI_CS_PORT4: now also J2.33 (GPIO11)
- net SPI_CS_PORT5: now also J2.35 (GPIO10)
- net SPI_CS_PORT6: now also J2.37 (GPIO9)
- net SPI_CS_PORT7: now also J2.39 (GPIO8)
- net SPI_MISO: now also J2.49 (GPIO4)
- net SPI_MOSI: now also J2.43 (GPIO7)
- net TCT: now also J2.40 (TCT)
- net TD+: now also J2.34 (ETH_TD+)
- net TD-: now also J2.36 (ETH_TD-)
- net USB_RP_D+: now also J2.69 (USB_D+)
- net USB_RP_D-: now also J2.71 (USB_D-)
- net VBUS: now also J2.72 (VBUS), J2.74 (VBUS), J2.75 (VBUS)

Commit message: finalized 1.0.0 revision, PCB, PCBA ordered
Parts:
- C18, C19: footprint Capacitor_SMD:C_0402_1005Metric -> DS_Capacitor:C_0402_1005Metric
- J2: now in the parts list
Connections:
- net SPI_CS: now reaches J2.47 (GPIO5)
Changed lines of the file:
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@@
+	(wire
+		(pts
+			(xy 151.13 135.89) (xy 172.72 135.89)
+		)
+		(stroke
+			(width 0)
+			(type default)
+		)
+	)
 	(wire
 		(pts
@@
 			)
 			(justify left)
+		)
+	)
+	(hierarchical_label "SPI_CS"
+		(shape output)
+		(at 151.13 135.89 180)
+		(effects
+			(font
+				(size 1.27 1.27)
+			)
+			(justify right)
 		)
 	)
@@
 			)
 		)
-		(property "Footprint" "Capacitor_SMD:C_0402_1005Metric"
+		(property "Footprint" "DS_Capacitor:C_0402_1005Metric"
 			(at 35.56 249.174 0)
 			(show_name yes)
@@
 		(unit 1)
 		(exclude_from_sim yes)
-		(in_bom no)
+		(in_bom yes)
 		(on_board yes)
 		(dnp no)
@@
 			)
 		)
-		(property "Footprint" "Capacitor_SMD:C_0402_1005Metric"
+		(property "Footprint" "DS_Capacitor:C_0402_1005Metric"
 			(at 54.61 249.174 0)
 			(show_name yes)

Commit message: minor fixes, start with software
Parts:
- added R31: 2.2K 5%, DS_Resistor:R_Array_Convex_4x0603, symbol DS_Resistor_1206:2.2K 5% ARRAY 1206
Connections:
- net +3.3V: now also R31.5 (R24), R31.6 (R23), R31.7 (R22), R31.8 (R12)
- net I2C1_SCL: now also R31.4 (R14)
- net I2C1_SDA: now also R31.3 (R13)
- no-connect marks 1 -> 3
