File: src/HardwareDesign/1.0.0/PDNode-600_Pro_Baseboard_100/external_power_connectors.kicad_sch (KiCad schematic)
At the start: 5 parts

Commit message: M54 rework
Other:
- company: DvidMakesThings -> ${COMPANY}
- moved on the sheet: H1, H2, H3, H4, H5
Changed lines of the file:
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@@
 	(title_block
 		(title "External Power Connectors")
-		(date "2026-02-05")
-		(rev "1.0.0")
-		(company "DvidMakesThings")
+		(date "2025-01-12")
+		(rev "${REVISION}")
+		(company "${COMPANY}")
 	)
 	(text "MOUNTING HOLES"
 		(exclude_from_sim no)
-		(at 23.368 196.342 0)
+		(at 33.528 196.342 0)
 		(effects
 			(font
@@
 	)
 	(junction
-		(at 55.88 233.68)
+		(at 66.04 233.68)
 		(diameter 0)
 		(color 0 0 0 0)
 	)
 	(junction
-		(at 55.88 254)
+		(at 66.04 254)
 		(diameter 0)
 		(color 0 0 0 0)
 	)
 	(junction
-		(at 55.88 243.84)
+		(at 66.04 243.84)
 		(diameter 0)
 		(color 0 0 0 0)
 	)
 	(junction
-		(at 55.88 223.52)
+		(at 66.04 223.52)
 		(diameter 0)
 		(color 0 0 0 0)
@@
 	(wire
 		(pts
-			(xy 48.26 243.84) (xy 55.88 243.84)
-		)
-		(stroke
-			(width 0)
-			(type default)
-		)
-	)
-	(wire
-		(pts
-			(xy 48.26 223.52) (xy 55.88 223.52)
-		)
-		(stroke
-			(width 0)
-			(type default)
-		)
-	)
-	(wire
-		(pts
-			(xy 55.88 254) (xy 55.88 259.08)
-		)
-		(stroke
-			(width 0)
-			(type default)
-		)
-	)
-	(wire
-		(pts
-			(xy 48.26 233.68) (xy 55.88 233.68)
-		)
-		(stroke
-			(width 0)
-			(type default)
-		)
-	)
-	(wire
-		(pts
-			(xy 48.26 254) (xy 55.88 254)
-		)
-		(stroke
-			(width 0)
-			(type default)
-		)
-	)
-	(wire
-		(pts
-			(xy 55.88 233.68) (xy 55.88 243.84)
-		)
-		(stroke
-			(width 0)
-			(type default)
-		)
-	)
-	(wire
-		(pts
-			(xy 48.26 213.36) (xy 55.88 213.36)
-		)
-		(stroke
-			(width 0)
-			(type default)
-		)
-	)
-	(wire
-		(pts
-			(xy 55.88 213.36) (xy 55.88 223.52)
-		)
-		(stroke
-			(width 0)
-			(type default)
-		)
-	)
-	(wire
-		(pts
-			(xy 55.88 254) (xy 55.88 243.84)
-		)
-		(stroke
-			(width 0)
-			(type default)
-		)
-	)
-	(wire
-		(pts
-			(xy 55.88 223.52) (xy 55.88 233.68)
+			(xy 58.42 243.84) (xy 66.04 243.84)
+		)
+		(stroke
+			(width 0)
+			(type default)
+		)
+	)
+	(wire
+		(pts
+			(xy 58.42 223.52) (xy 66.04 223.52)
+		)
+		(stroke
+			(width 0)
+			(type default)
+		)
+	)
+	(wire
+		(pts
+			(xy 66.04 254) (xy 66.04 259.08)
+		)
+		(stroke
+			(width 0)
+			(type default)
+		)
+	)
+	(wire
+		(pts
+			(xy 58.42 233.68) (xy 66.04 233.68)
+		)
+		(stroke
+			(width 0)
+			(type default)
+		)
+	)
+	(wire
+		(pts
+			(xy 58.42 254) (xy 66.04 254)
+		)
+		(stroke
+			(width 0)
+			(type default)
+		)
+	)
+	(wire
+		(pts
+			(xy 66.04 233.68) (xy 66.04 243.84)
+		)
+		(stroke
+			(width 0)
+			(type default)
+		)
+	)
+	(wire
+		(pts
+			(xy 58.42 213.36) (xy 66.04 213.36)
+		)
+		(stroke
+			(width 0)
+			(type default)
+		)
+	)
+	(wire
+		(pts
+			(xy 66.04 213.36) (xy 66.04 223.52)
+		)
+		(stroke
+			(width 0)
+			(type default)
+		)
+	)
+	(wire
+		(pts
+			(xy 66.04 254) (xy 66.04 243.84)
+		)
+		(stroke
+			(width 0)
+			(type default)
+		)
+	)
+	(wire
+		(pts
+			(xy 66.04 223.52) (xy 66.04 233.68)
 		)
 		(stroke
@@
 	(symbol
 		(lib_id "Mechanical:MountingHole_Pad")
-		(at 45.72 254 90)
+		(at 55.88 254 90)
 		(unit 1)
 		(exclude_from_sim no)
@@
 		(fields_autoplaced yes)
 		(property "Reference" "H5"
-			(at 44.45 247.65 90)
+			(at 54.61 247.65 90)
 			(effects
 				(font
@@
 		)
 		(property "Value" "MountingHole_Pad"
-			(at 44.45 250.19 90)
+			(at 54.61 250.19 90)
 			(effects
 				(font
@@
 		)
 		(property "Footprint" "MountingHole:MountingHole_3.2mm_M3_Pad_Via"
-			(at 45.72 254 0)
+			(at 55.88 254 0)
 			(effects
 				(font
@@
 		)
 		(property "Datasheet" "~"
-			(at 45.72 254 0)
+			(at 55.88 254 0)
 			(effects
 				(font
@@
 		)
 		(property "Description" "Mounting Hole with connection"
-			(at 45.72 254 0)
+			(at 55.88 254 0)
 			(effects
 				(font
@@
 	(symbol
 		(lib_id "Mechanical:MountingHole_Pad")
-		(at 45.72 243.84 90)
+		(at 55.88 243.84 90)
 		(unit 1)
 		(exclude_from_sim no)
@@
 		(fields_autoplaced yes)
 		(property "Reference" "H4"
-			(at 44.45 237.49 90)
+			(at 54.61 237.49 90)
 			(effects
 				(font
@@
 		)
 		(property "Value" "MountingHole_Pad"
-			(at 44.45 240.03 90)
+			(at 54.61 240.03 90)
 			(effects
 				(font
@@
 		)
 		(property "Footprint" "MountingHole:MountingHole_3.2mm_M3_Pad_Via"
-			(at 45.72 243.84 0)
+			(at 55.88 243.84 0)
 			(effects
 				(font
@@
 		)
 		(property "Datasheet" "~"
-			(at 45.72 243.84 0)
+			(at 55.88 243.84 0)
 			(effects
 				(font
@@
 		)
 		(property "Description" "Mounting Hole with connection"
-			(at 45.72 243.84 0)
+			(at 55.88 243.84 0)
 			(effects
 				(font
@@
 	(symbol
 		(lib_id "DS_Supply:SHIELD")
-		(at 55.88 260.35 0)
+		(at 66.04 260.35 0)
 		(mirror y)
 		(unit 1)
@@
 		(fields_autoplaced yes)
 		(property "Reference" "#SHIELD05"
-			(at 55.88 251.46 0)
+			(at 66.04 251.46 0)
 			(effects
 				(font
@@
 		)
 		(property "Value" "SHIELD"
-			(at 53.34 260.8579 0)
+			(at 63.5 260.8579 0)
 			(effects
 				(font
@@
 		)
 		(property "Footprint" ""
-			(at 55.88 260.35 0)
+			(at 66.04 260.35 0)
 			(effects
 				(font
@@
 		)
 		(property "Datasheet" ""
-			(at 55.88 260.35 0)
+			(at 66.04 260.35 0)
 			(effects
 				(font
@@
 		)
 		(property "Description" "Power symbol creates a global label with name \"SHIELD\""
-			(at 55.372 253.238 0)
+			(at 65.532 253.238 0)
 			(effects
 				(font
@@
 	(symbol
 		(lib_id "Mechanical:MountingHole_Pad")
-		(at 45.72 223.52 90)
+		(at 55.88 223.52 90)
 		(unit 1)
 		(exclude_from_sim no)
@@
 		(fields_autoplaced yes)
 		(property "Reference" "H2"
-			(at 44.45 217.17 90)
+			(at 54.61 217.17 90)
 			(effects
 				(font
@@
 		)
 		(property "Value" "MountingHole_Pad"
-			(at 44.45 219.71 90)
+			(at 54.61 219.71 90)
 			(effects
 				(font
@@
 		)
 		(property "Footprint" "MountingHole:MountingHole_3.2mm_M3_Pad_Via"
-			(at 45.72 223.52 0)
+			(at 55.88 223.52 0)
 			(effects
 				(font
@@
 		)
 		(property "Datasheet" "~"
-			(at 45.72 223.52 0)
+			(at 55.88 223.52 0)
 			(effects
 				(font
@@
 		)
 		(property "Description" "Mounting Hole with connection"
-			(at 45.72 223.52 0)
+			(at 55.88 223.52 0)
 			(effects
 				(font
@@
 	(symbol
 		(lib_id "Mechanical:MountingHole_Pad")
-		(at 45.72 213.36 90)
+		(at 55.88 213.36 90)
 		(unit 1)
 		(exclude_from_sim no)
@@
 		(fields_autoplaced yes)
 		(property "Reference" "H1"
-			(at 44.45 207.01 90)
+			(at 54.61 207.01 90)
 			(effects
 				(font
@@
 		)
 		(property "Value" "MountingHole_Pad"
-			(at 44.45 209.55 90)
+			(at 54.61 209.55 90)
 			(effects
 				(font
@@
 		)
 		(property "Footprint" "MountingHole:MountingHole_3.2mm_M3_Pad_Via"
-			(at 45.72 213.36 0)
+			(at 55.88 213.36 0)
 			(effects
 				(font
@@
 		)
 		(property "Datasheet" "~"
-			(at 45.72 213.36 0)
+			(at 55.88 213.36 0)
 			(effects
 				(font
@@
 		)
 		(property "Description" "Mounting Hole with connection"
-			(at 45.72 213.36 0)
+			(at 55.88 213.36 0)
 			(effects
 				(font
@@
 	(symbol
 		(lib_id "Mechanical:MountingHole_Pad")
-		(at 45.72 233.68 90)
+		(at 55.88 233.68 90)
 		(unit 1)
 		(exclude_from_sim no)
@@
 		(fields_autoplaced yes)
 		(property "Reference" "H3"
-			(at 44.45 227.33 90)
+			(at 54.61 227.33 90)
 			(effects
 				(font
@@
 		)
 		(property "Value" "MountingHole_Pad"
-			(at 44.45 229.87 90)
+			(at 54.61 229.87 90)
 			(effects
 				(font
@@
 		)
 		(property "Footprint" "MountingHole:MountingHole_3.2mm_M3_Pad_Via"
-			(at 45.72 233.68 0)
+			(at 55.88 233.68 0)
 			(effects
 				(font
@@
 		)
 		(property "Datasheet" "~"
-			(at 45.72 233.68 0)
+			(at 55.88 233.68 0)
 			(effects
 				(font
@@
 		)
 		(property "Description" "Mounting Hole with connection"
-			(at 45.72 233.68 0)
-			(effects
-				(font
+			(at 55.88 233.68 0)
+			(effects
+				(font

Commit message: baseboard development
Parts:
- added C67: 330uF 50V, DS_Capacitor:CP_Elec_10x10.5, symbol DS_Capacitor_ELKO:330uF 50V
- added C68: 100nF 50V, Capacitor_SMD:C_0402_1005Metric, symbol DS_Capacitor_0402:100nF 50V 0402
- added F1: 0ATO030.VP, DS_Fuse:178.6165.0001-Littelfuse, symbol DS_Fuse:0ATO030.VP
- added J22: 1724470208, DS_Connector:MOLEX_1724470208, symbol DS_Connector:Molex 8 Pin (2x4) PC header
- added R29: 51K 1%, Resistor_SMD:R_0402_1005Metric, symbol DS_Resistor_0402:51K_1%
- added R30: 5.1K 1%, Resistor_SMD:R_0402_1005Metric, symbol DS_Resistor_0402:5.1K 1% 0402
Connections:
- new net +24V: C67.1, F1.5 (F1), F1.6 (F1), F1.7 (F1), F1.8 (F1), R29.1
- new net +24V_IN: F1.1 (F2), F1.2 (F2), F1.3 (F2), F1.4 (F2), J22.5, J22.6, J22.7, J22.8
- new net ADC_24V: C68.1, R29.2, R30.1
- new net GND: C67.2, C68.2, J22.1, J22.2, J22.3, J22.4, R30.2
Other:
- note added: "1724470208 Datasheet: Current - Maximum per Contact 9.0A"
- note added: "32V 30A Blade Fuse"
- note added: "8 PIN EPS +24V POWER CONNECTOR"
- moved on the sheet: H1, H2, H3, H4, H5

Commit message: update readme, add documentation
Other:
- moved on the sheet: C67, C68, F1, H1, H2, H3, H4, H5, J22, R29, R30

Commit message: finalized 1.0.0 revision, PCB, PCBA ordered
Parts:
- C68: footprint Capacitor_SMD:C_0402_1005Metric -> DS_Capacitor:C_0402_1005Metric
- R29, R30: footprint Resistor_SMD:R_0402_1005Metric -> DS_Resistor:R_0402_1005Metric
Changed lines of the file:
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@@
 			)
 		)
-		(property "Footprint" "Resistor_SMD:R_0402_1005Metric"
+		(property "Footprint" "DS_Resistor:R_0402_1005Metric"
 			(at 256.032 136.144 0)
 			(effects
@@
 			)
 		)
-		(property "Footprint" "Resistor_SMD:R_0402_1005Metric"
+		(property "Footprint" "DS_Resistor:R_0402_1005Metric"
 			(at 256.032 123.444 0)
 			(effects
@@
 			)
 		)
-		(property "Footprint" "Capacitor_SMD:C_0402_1005Metric"
+		(property "Footprint" "DS_Capacitor:C_0402_1005Metric"
 			(at 274.32 136.144 0)
 			(show_name yes)
