File: src/HardwareDesign/1.0.0/PDNode-600_Pro_Baseboard_100/pdc_signals.kicad_sch (KiCad schematic)
At the start: 24 parts, among them IC10 SN74LVC1G97QDCKRQ1, IC11 SN74LVC1G97QDCKRQ1, IC12 SN74LVC1G97QDCKRQ1, IC13 SN74LVC1G97QDCKRQ1, IC14 MCP23017T-E/ML, IC15 MCP23017T-E/ML, IC16 MCP23017T-E/ML, IC5 SN74LVC1G97QDCKRQ1, IC6 SN74LVC1G97QDCKRQ1, IC7 SN74LVC1G97QDCKRQ1, IC8 SN74LVC1G97QDCKRQ1, IC9 MCP23017T-E/ML

Commit message: M54 rework
Other:
- company: DvidMakesThings -> ${COMPANY}
Changed lines of the file:
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@@
 	(title_block
 		(title "PDC Signals")
-		(date "2026-02-05")
-		(rev "1.0.0")
-		(company "DvidMakesThings")
+		(date "2025-01-12")
+		(rev "${REVISION}")
+		(company "${COMPANY}")
 	)
 	(text "Read expander: A2=0, A1=1, A0=1 -> 0x23"

Commit message: finalized 1.0.0 revision, PCB, PCBA ordered
Parts:
- C24, C25, C26, C27, C28, C29, C30, C31, C32, C33, C34, C35: footprint Capacitor_SMD:C_0402_1005Metric -> DS_Capacitor:C_0402_1005Metric
Changed lines of the file:
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@@
 			)
 		)
-		(property "Footprint" "Capacitor_SMD:C_0402_1005Metric"
+		(property "Footprint" "DS_Capacitor:C_0402_1005Metric"
 			(at 304.8 109.474 0)
 			(show_name yes)
@@
 			)
 		)
-		(property "Footprint" "Capacitor_SMD:C_0402_1005Metric"
+		(property "Footprint" "DS_Capacitor:C_0402_1005Metric"
 			(at 102.87 264.414 0)
 			(show_name yes)
@@
 			)
 		)
-		(property "Footprint" "Capacitor_SMD:C_0402_1005Metric"
+		(property "Footprint" "DS_Capacitor:C_0402_1005Metric"
 			(at 173.99 264.414 0)
 			(show_name yes)
@@
 			)
 		)
-		(property "Footprint" "Capacitor_SMD:C_0402_1005Metric"
+		(property "Footprint" "DS_Capacitor:C_0402_1005Metric"
 			(at 289.56 209.804 0)
 			(show_name yes)
@@
 			)
 		)
-		(property "Footprint" "Capacitor_SMD:C_0402_1005Metric"
+		(property "Footprint" "DS_Capacitor:C_0402_1005Metric"
 			(at 67.31 264.414 0)
 			(show_name yes)
@@
 			)
 		)
-		(property "Footprint" "Capacitor_SMD:C_0402_1005Metric"
+		(property "Footprint" "DS_Capacitor:C_0402_1005Metric"
 			(at 49.53 264.414 0)
 			(show_name yes)
@@
 			)
 		)
-		(property "Footprint" "Capacitor_SMD:C_0402_1005Metric"
+		(property "Footprint" "DS_Capacitor:C_0402_1005Metric"
 			(at 85.09 264.414 0)
 			(show_name yes)
@@
 			)
 		)
-		(property "Footprint" "Capacitor_SMD:C_0402_1005Metric"
+		(property "Footprint" "DS_Capacitor:C_0402_1005Metric"
 			(at 156.21 264.414 0)
 			(show_name yes)
@@
 			)
 		)
-		(property "Footprint" "Capacitor_SMD:C_0402_1005Metric"
+		(property "Footprint" "DS_Capacitor:C_0402_1005Metric"
 			(at 120.65 264.414 0)
 			(show_name yes)
@@
 			)
 		)
-		(property "Footprint" "Capacitor_SMD:C_0402_1005Metric"
+		(property "Footprint" "DS_Capacitor:C_0402_1005Metric"
 			(at 138.43 264.414 0)
 			(show_name yes)
@@
 			)
 		)
-		(property "Footprint" "Capacitor_SMD:C_0402_1005Metric"
+		(property "Footprint" "DS_Capacitor:C_0402_1005Metric"
 			(at 33.02 195.834 0)
 			(show_name yes)
@@
 			)
 		)
-		(property "Footprint" "Capacitor_SMD:C_0402_1005Metric"
+		(property "Footprint" "DS_Capacitor:C_0402_1005Metric"
 			(at 157.48 195.834 0)
 			(show_name yes)
