File: src/HardwareDesign/1.0.0/PDNode-600_Pro_Baseboard_100/pdcard_connectors_5-8.kicad_sch (KiCad schematic)
At the start: 12 parts, among them J10 10018784-10200TLF, J11 10018784-10200TLF, J8 10018784-10200TLF, J9 10018784-10200TLF

Commit message: M54 rework
Other:
- company: DvidMakesThings -> ${COMPANY}
Changed lines of the file:
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@@
 	(title_block
 		(title "PDCard Connectors 5-8")
-		(date "2026-02-05")
-		(rev "1.0.0")
-		(company "DvidMakesThings")
+		(date "2025-01-12")
+		(rev "${REVISION}")
+		(company "${COMPANY}")
 	)
 	(text "A9 is used as card detected.\nPull B9 on the Baseboard to GND with 10K\n-> 0 = not connected, 1 = connected"

Commit message: finalized 1.0.0 revision, PCB, PCBA ordered
Parts:
- R52, R53, R54, R55: footprint Resistor_SMD:R_0402_1005Metric -> DS_Resistor:R_0402_1005Metric
Changed lines of the file:
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@@
 			)
 		)
-		(property "Footprint" "Resistor_SMD:R_0402_1005Metric"
+		(property "Footprint" "DS_Resistor:R_0402_1005Metric"
 			(at 339.852 211.074 0)
 			(effects
@@
 			)
 		)
-		(property "Footprint" "Resistor_SMD:R_0402_1005Metric"
+		(property "Footprint" "DS_Resistor:R_0402_1005Metric"
 			(at 341.122 112.014 0)
 			(effects
@@
 			)
 		)
-		(property "Footprint" "Resistor_SMD:R_0402_1005Metric"
+		(property "Footprint" "DS_Resistor:R_0402_1005Metric"
 			(at 158.242 112.014 0)
 			(effects
@@
 			)
 		)
-		(property "Footprint" "Resistor_SMD:R_0402_1005Metric"
+		(property "Footprint" "DS_Resistor:R_0402_1005Metric"
 			(at 156.972 211.074 0)
 			(effects
