File: src/HardwareDesign/1.0.0/PDNode-600_Pro_Baseboard_100/system_power.kicad_sch (KiCad schematic)
At the start: 43 parts, among them IC1 TPS51225CRUKR, T1 FDMC7692, T2 FDMC7692, T3 FDMC7672, T4 FDMC7672

Commit message: M54 rework
Other:
- company: DvidMakesThings -> ${COMPANY}
Changed lines of the file:
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@@
 	(title_block
 		(title "System Power")
-		(date "2026-02-05")
-		(rev "1.0.0")
-		(company "DvidMakesThings")
+		(date "2025-01-12")
+		(rev "${REVISION}")
+		(company "${COMPANY}")
 	)
 	(text "+3.3V 100mA OUTPUT"

Commit message: finalized 1.0.0 revision, PCB, PCBA ordered
Parts:
- C12, C13, C14, C15, C16, C17, C7, C8: footprint Capacitor_SMD:C_0402_1005Metric -> DS_Capacitor:C_0402_1005Metric
- C2, C3, C4, C5, C6: footprint Capacitor_SMD:C_0805_2012Metric -> DS_Capacitor:C_0805_2012Metric
- R10, R11, R12, R13, R14, R15, R16, R17, R18, R19, R2, R5, R6, R7, R8, R9: footprint Resistor_SMD:R_0402_1005Metric -> DS_Resistor:R_0402_1005Metric
- R3, R4: footprint Resistor_SMD:R_0402_1005Metric -> DS_Resistor:R_0402_1005Metric; LCSC_PART C25101 -> C2909330
Changed lines of the file:
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@@
 			)
 		)
-		(property "Footprint" "Resistor_SMD:R_0402_1005Metric"
+		(property "Footprint" "DS_Resistor:R_0402_1005Metric"
 			(at 214.122 190.754 0)
 			(effects
@@
 			)
 		)
-		(property "Footprint" "Capacitor_SMD:C_0805_2012Metric"
+		(property "Footprint" "DS_Capacitor:C_0805_2012Metric"
 			(at 107.95 81.534 0)
 			(show_name yes)
@@
 			)
 		)
-		(property "Footprint" "Resistor_SMD:R_0402_1005Metric"
+		(property "Footprint" "DS_Resistor:R_0402_1005Metric"
 			(at 214.122 175.514 0)
 			(effects
@@
 			)
 		)
-		(property "Footprint" "Resistor_SMD:R_0402_1005Metric"
+		(property "Footprint" "DS_Resistor:R_0402_1005Metric"
 			(at 245.872 190.754 0)
 			(effects
@@
 			)
 		)
-		(property "Footprint" "Resistor_SMD:R_0402_1005Metric"
+		(property "Footprint" "DS_Resistor:R_0402_1005Metric"
 			(at 290.322 123.444 0)
 			(effects
@@
 			)
 		)
-		(property "Footprint" "Resistor_SMD:R_0402_1005Metric"
+		(property "Footprint" "DS_Resistor:R_0402_1005Metric"
 			(at 90.932 108.204 0)
 			(effects
@@
 			)
 		)
-		(property "Footprint" "Resistor_SMD:R_0402_1005Metric"
+		(property "Footprint" "DS_Resistor:R_0402_1005Metric"
 			(at 141.732 122.174 0)
 			(effects
@@
 			)
 		)
-		(property "Footprint" "Capacitor_SMD:C_0402_1005Metric"
+		(property "Footprint" "DS_Capacitor:C_0402_1005Metric"
 			(at 124.46 159.004 0)
 			(show_name yes)
@@
 			)
 		)
-		(property "Footprint" "Capacitor_SMD:C_0805_2012Metric"
+		(property "Footprint" "DS_Capacitor:C_0805_2012Metric"
 			(at 332.74 81.534 0)
 			(show_name yes)
@@
 			)
 		)
-		(property "Footprint" "Resistor_SMD:R_0402_1005Metric"
+		(property "Footprint" "DS_Resistor:R_0402_1005Metric"
 			(at 182.372 190.754 0)
 			(effects
@@
 			)
 		)
-		(property "Footprint" "Resistor_SMD:R_0402_1005Metric"
+		(property "Footprint" "DS_Resistor:R_0402_1005Metric"
 			(at 273.812 175.514 0)
 			(effects
@@
 			)
 		)
-		(property "Footprint" "Resistor_SMD:R_0402_1005Metric"
+		(property "Footprint" "DS_Resistor:R_0402_1005Metric"
 			(at 255.524 83.058 0)
 			(effects
@@
 			)
 		)
-		(property "Datasheet" ""
+		(property "Datasheet" "https://jlcpcb.com/api/file/downloadByFileSystemAccessId/8590208205541711872"
 			(at 266.446 83.058 0)
 			(show_name yes)
@@
 			)
 		)
-		(property "LCSC_PART" "C25101"
+		(property "LCSC_PART" "C2909330"
 			(at 264.414 83.058 0)
 			(show_name yes)
@@
 			)
 		)
-		(property "Footprint" "Resistor_SMD:R_0402_1005Metric"
+		(property "Footprint" "DS_Resistor:R_0402_1005Metric"
 			(at 330.962 123.444 0)
 			(effects
@@
 			)
 		)
-		(property "Footprint" "Capacitor_SMD:C_0805_2012Metric"
+		(property "Footprint" "DS_Capacitor:C_0805_2012Metric"
 			(at 177.8 80.264 0)
 			(show_name yes)
@@
 			)
 		)
-		(property "Footprint" "Capacitor_SMD:C_0805_2012Metric"
+		(property "Footprint" "DS_Capacitor:C_0805_2012Metric"
 			(at 350.52 81.534 0)
 			(show_name yes)
@@
 			)
 		)
-		(property "Footprint" "Capacitor_SMD:C_0402_1005Metric"
+		(property "Footprint" "DS_Capacitor:C_0402_1005Metric"
 			(at 146.05 159.004 0)
 			(show_name yes)
@@
 			)
 		)
-		(property "Footprint" "Capacitor_SMD:C_0805_2012Metric"
+		(property "Footprint" "DS_Capacitor:C_0805_2012Metric"
 			(at 90.17 81.534 0)
 			(show_name yes)
@@
 			)
 		)
-		(property "Footprint" "Capacitor_SMD:C_0402_1005Metric"
+		(property "Footprint" "DS_Capacitor:C_0402_1005Metric"
 			(at 241.554 81.28 0)
 			(show_name yes)
@@
 			)
 		)
-		(property "Footprint" "Resistor_SMD:R_0402_1005Metric"
+		(property "Footprint" "DS_Resistor:R_0402_1005Metric"
 			(at 330.962 110.744 0)
 			(effects
@@
 			)
 		)
-		(property "Footprint" "Capacitor_SMD:C_0402_1005Metric"
+		(property "Footprint" "DS_Capacitor:C_0402_1005Metric"
 			(at 234.95 134.874 0)
 			(show_name yes)
@@
 			)
 		)
-		(property "Footprint" "Resistor_SMD:R_0402_1005Metric"
+		(property "Footprint" "DS_Resistor:R_0402_1005Metric"
 			(at 245.872 175.514 0)
 			(effects
@@
 			)
 		)
-		(property "Footprint" "Capacitor_SMD:C_0402_1005Metric"
+		(property "Footprint" "DS_Capacitor:C_0402_1005Metric"
 			(at 135.89 178.054 0)
 			(show_name yes)
@@
 			)
 		)
-		(property "Footprint" "Resistor_SMD:R_0402_1005Metric"
+		(property "Footprint" "DS_Resistor:R_0402_1005Metric"
 			(at 176.022 133.604 0)
 			(effects
@@
 			)
 		)
-		(property "Footprint" "Resistor_SMD:R_0402_1005Metric"
+		(property "Footprint" "DS_Resistor:R_0402_1005Metric"
 			(at 267.462 80.264 0)
 			(effects
@@
 			)
 		)
-		(property "Footprint" "Resistor_SMD:R_0402_1005Metric"
+		(property "Footprint" "DS_Resistor:R_0402_1005Metric"
 			(at 90.932 120.904 0)
 			(effects
@@
 			)
 		)
-		(property "Footprint" "Resistor_SMD:R_0402_1005Metric"
+		(property "Footprint" "DS_Resistor:R_0402_1005Metric"
 			(at 273.812 190.754 0)
 			(effects
@@
 			)
 		)
-		(property "Footprint" "Resistor_SMD:R_0402_1005Metric"
+		(property "Footprint" "DS_Resistor:R_0402_1005Metric"
 			(at 182.372 175.514 0)
 			(effects
@@
 			)
 		)
-		(property "Footprint" "Capacitor_SMD:C_0402_1005Metric"
+		(property "Footprint" "DS_Capacitor:C_0402_1005Metric"
 			(at 114.3 178.054 0)
 			(show_name yes)
@@
 			)
 		)
-		(property "Footprint" "Capacitor_SMD:C_0402_1005Metric"
+		(property "Footprint" "DS_Capacitor:C_0402_1005Metric"
 			(at 180.086 86.36 0)
 			(show_name yes)
@@
 			)
 		)
-		(property "Footprint" "Capacitor_SMD:C_0402_1005Metric"
+		(property "Footprint" "DS_Capacitor:C_0402_1005Metric"
 			(at 191.77 134.874 0)
 			(show_name yes)
@@
 			)
 		)
-		(property "Footprint" "Resistor_SMD:R_0402_1005Metric"
+		(property "Footprint" "DS_Resistor:R_0402_1005Metric"
 			(at 163.576 88.138 0)
 			(effects
@@
 			)
 		)
-		(property "Datasheet" ""
+		(property "Datasheet" "https://jlcpcb.com/api/file/downloadByFileSystemAccessId/8590208205541711872"
 			(at 152.654 88.138 0)
 			(show_name yes)
@@
 			)
 		)
-		(property "LCSC_PART" "C25101"
+		(property "LCSC_PART" "C2909330"
 			(at 154.686 88.138 0)
 			(show_name yes)

Commit message: minor fixes, start with software
Parts:
- removed C12, C13: 1nF 50V, DS_Capacitor:C_0402_1005Metric, symbol DS_Capacitor_0402:1nF 50V 0402
- added C12, C13: 2.2uF 25V, DS_Capacitor:C_0402_1005Metric, symbol DS_Capacitor_0402:2.2uF 25V 0402
Connections:
- net +3.3VA: now also C13.1
- net +5VA: now also C12.1
- net GND: now also C12.2, C13.2
