File: src/HardwareDesign/1.0.0/PDNode-600_Pro_Baseboard_100/usb_interface.kicad_sch (KiCad schematic)
At the start: 13 parts, among them IC3 FSUSB42MUX, J3 USB-TYPE-C-018

Commit message: M54 rework
Other:
- company: DvidMakesThings -> ${COMPANY}
Changed lines of the file:
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@@
 	(title_block
 		(title "USB Interface")
-		(date "2026-02-05")
-		(rev "1.0.0")
-		(company "DvidMakesThings")
+		(date "2025-01-12")
+		(rev "${REVISION}")
+		(company "${COMPANY}")
 	)
 	(text "USB DATA-PATH SELECTOR"

Commit message: baseboard development
Parts:
- removed C22: 100nF 50V, Capacitor_SMD:C_0402_1005Metric, symbol DS_Capacitor_0402:100nF 50V 0402
- removed IC3: FSUSB42MUX, DS_Peripherals:MSOP-10_3x3mm_P0.5mm, symbol DS_Peripherals:FSUSB42MUX
- removed R20: 5.1K 1%, Resistor_SMD:R_0402_1005Metric, symbol DS_Resistor_0402:5.1K 1% 0402
Connections:
- net USB_D+ is gone; now on net USB_RP_D+: D4.2, J3.A6 (D+), J3.B6 (D+)
- net USB_D- is gone; now on net USB_RP_D-: D4.3, J3.A7 (D-), J3.B7 (D-)
Other:
- note added: "DISPLAY CONNECTOR"
- note removed: "For USB_RP lines, no TVS needed For USB_DBG lines, TVS is expected on the debug header itself"
- note removed: "OEn = 0 -> ENABLED SEL = 0 -> HSD1+/- SEL = 1 -> HSD2+/-"
- note removed: "The purpose of the MUX is debugging. By default SEL = 0, it's connecting to the MCU Attaching the debug header will pull SEL to 1 and USB route is redirected"
- note removed: "USB DATA-PATH SELECTOR"
- moved on the sheet: C20, C21, C23, D4, D5, J3, R21, R22, R23, R24

Commit message: finalized 1.0.0 revision, PCB, PCBA ordered
Parts:
- added J23: 0525592052, DS_Connector:CON_525592052_MOL, symbol DS_Connector:20P-FPC
- C20, C21: footprint Capacitor_SMD:C_0402_1005Metric -> DS_Capacitor:C_0402_1005Metric
- C23: footprint Capacitor_SMD:C_1206_3216Metric -> DS_Capacitor:C_1206_3216Metric
- D5: footprint LED_SMD:LED_0402_1005Metric -> DS_Opto:LED_0402_1005Metric
- R21, R22, R24: footprint Resistor_SMD:R_0402_1005Metric -> DS_Resistor:R_0402_1005Metric
- R23: footprint Resistor_SMD:R_1206_3216Metric -> DS_Resistor:R_1206_3216Metric
Connections:
- net GND: now also J23.1, J23.10, J23.12, J23.14, J23.15, J23.16, J23.18, J23.20
- net SHIELD: now also J23.P1, J23.P2, J23.P3, J23.P4
- new net +3.3V: J23.2, J23.4, J23.6
- new net +5V: J23.3, J23.5, J23.8
- new net I2C1_SCL: J23.17
- new net I2C1_SDA: J23.19
- new net SPI_CLK: J23.9
- new net SPI_CS: J23.11
- new net SPI_MISO: J23.13
- new net SPI_MOSI: J23.7
