File: src/HardwareDesign/1.0.0/PDNode-600_Pro_Baseboard_100/usba_current_measurement.kicad_sch (KiCad schematic)
At the start: 50 parts, among them IC21 SN74LVC1G97QDCKRQ1, IC22 PAC1720-1-AIA-TR, IC23 SN74LVC1G97QDCKRQ1, IC24 PAC1720-1-AIA-TR, IC25 SN74LVC1G97QDCKRQ1, IC26 SN74LVC1G97QDCKRQ1, IC27 MCP23017T-E/ML, J14 Conn_01x02, J15 Conn_01x02, J16 Conn_01x02, J17 Conn_01x02, J18 Conn_01x02, J19 Conn_01x02, J20 Conn_01x02, J21 Conn_01x02

Commit message: M54 rework
Other:
- company: DvidMakesThings -> ${COMPANY}
Changed lines of the file:
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@@
 	(title_block
 		(title "USB-A Current Measurement")
-		(date "2026-02-05")
-		(rev "1.0.0")
-		(company "DvidMakesThings")
+		(date "2025-01-12")
+		(rev "${REVISION}")
+		(company "${COMPANY}")
 	)
 	(text "Place 10nF and 100R parts as physically \nclose to the PAC1720 pins as possible"

Commit message: finalized 1.0.0 revision, PCB, PCBA ordered
Parts:
- C54, C55, C56, C57, C58, C59, C60, C61, C62, C63, C65: footprint Capacitor_SMD:C_0402_1005Metric -> DS_Capacitor:C_0402_1005Metric
- R74, R75, R76, R77, R78, R79, R80, R81, R82, R83, R84, R85, R86, R87, R88, R89, R90, R91, R92, R93: footprint Resistor_SMD:R_0402_1005Metric -> DS_Resistor:R_0402_1005Metric
Changed lines of the file:
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@@
 			)
 		)
-		(property "Footprint" "Capacitor_SMD:C_0402_1005Metric"
+		(property "Footprint" "DS_Capacitor:C_0402_1005Metric"
 			(at 160.02 80.264 0)
 			(show_name yes)
@@
 			)
 		)
-		(property "Footprint" "Resistor_SMD:R_0402_1005Metric"
+		(property "Footprint" "DS_Resistor:R_0402_1005Metric"
 			(at 338.074 173.482 0)
 			(effects
@@
 			)
 		)
-		(property "Footprint" "Capacitor_SMD:C_0402_1005Metric"
+		(property "Footprint" "DS_Capacitor:C_0402_1005Metric"
 			(at 31.75 84.074 0)
 			(show_name yes)
@@
 			)
 		)
-		(property "Footprint" "Capacitor_SMD:C_0402_1005Metric"
+		(property "Footprint" "DS_Capacitor:C_0402_1005Metric"
 			(at 246.38 178.054 0)
 			(show_name yes)
@@
 			)
 		)
-		(property "Footprint" "Capacitor_SMD:C_0402_1005Metric"
+		(property "Footprint" "DS_Capacitor:C_0402_1005Metric"
 			(at 246.38 223.774 0)
 			(show_name yes)
@@
 			)
 		)
-		(property "Footprint" "Resistor_SMD:R_0402_1005Metric"
+		(property "Footprint" "DS_Resistor:R_0402_1005Metric"
 			(at 66.294 80.772 0)
 			(effects
@@
 			)
 		)
-		(property "Footprint" "Capacitor_SMD:C_0402_1005Metric"
+		(property "Footprint" "DS_Capacitor:C_0402_1005Metric"
 			(at 246.38 82.804 0)
 			(show_name yes)
@@
 			)
 		)
-		(property "Footprint" "Resistor_SMD:R_0402_1005Metric"
+		(property "Footprint" "DS_Resistor:R_0402_1005Metric"
 			(at 338.074 115.062 0)
 			(effects
@@
 			)
 		)
-		(property "Footprint" "Resistor_SMD:R_0402_1005Metric"
+		(property "Footprint" "DS_Resistor:R_0402_1005Metric"
 			(at 185.674 141.478 0)
 			(effects
@@
 			)
 		)
-		(property "Footprint" "Resistor_SMD:R_0402_1005Metric"
+		(property "Footprint" "DS_Resistor:R_0402_1005Metric"
 			(at 186.944 91.948 0)
 			(effects
@@
 			)
 		)
-		(property "Footprint" "Resistor_SMD:R_0402_1005Metric"
+		(property "Footprint" "DS_Resistor:R_0402_1005Metric"
 			(at 58.166 141.732 0)
 			(effects
@@
 			)
 		)
-		(property "Footprint" "Resistor_SMD:R_0402_1005Metric"
+		(property "Footprint" "DS_Resistor:R_0402_1005Metric"
 			(at 185.674 133.858 0)
 			(effects
@@
 			)
 		)
-		(property "Footprint" "Resistor_SMD:R_0402_1005Metric"
+		(property "Footprint" "DS_Resistor:R_0402_1005Metric"
 			(at 338.074 66.802 0)
 			(effects
@@
 			)
 		)
-		(property "Footprint" "Resistor_SMD:R_0402_1005Metric"
+		(property "Footprint" "DS_Resistor:R_0402_1005Metric"
 			(at 66.294 144.272 0)
 			(effects
@@
 			)
 		)
-		(property "Footprint" "Resistor_SMD:R_0402_1005Metric"
+		(property "Footprint" "DS_Resistor:R_0402_1005Metric"
 			(at 186.944 84.328 0)
 			(effects
@@
 			)
 		)
-		(property "Footprint" "Resistor_SMD:R_0402_1005Metric"
+		(property "Footprint" "DS_Resistor:R_0402_1005Metric"
 			(at 338.074 207.772 0)
 			(effects
@@
 			)
 		)
-		(property "Footprint" "Capacitor_SMD:C_0402_1005Metric"
+		(property "Footprint" "DS_Capacitor:C_0402_1005Metric"
 			(at 160.02 94.234 0)
 			(show_name yes)
@@
 			)
 		)
-		(property "Footprint" "Resistor_SMD:R_0402_1005Metric"
+		(property "Footprint" "DS_Resistor:R_0402_1005Metric"
 			(at 338.074 162.052 0)
 			(effects
@@
 			)
 		)
-		(property "Footprint" "Capacitor_SMD:C_0402_1005Metric"
+		(property "Footprint" "DS_Capacitor:C_0402_1005Metric"
 			(at 246.38 131.064 0)
 			(show_name yes)
@@
 			)
 		)
-		(property "Footprint" "Capacitor_SMD:C_0402_1005Metric"
+		(property "Footprint" "DS_Capacitor:C_0402_1005Metric"
 			(at 55.88 244.094 0)
 			(show_name yes)
@@
 			)
 		)
-		(property "Footprint" "Resistor_SMD:R_0402_1005Metric"
+		(property "Footprint" "DS_Resistor:R_0402_1005Metric"
 			(at 186.944 77.978 0)
 			(effects
@@
 			)
 		)
-		(property "Footprint" "Resistor_SMD:R_0402_1005Metric"
+		(property "Footprint" "DS_Resistor:R_0402_1005Metric"
 			(at 338.074 126.492 0)
 			(effects
@@
 			)
 		)
-		(property "Footprint" "Resistor_SMD:R_0402_1005Metric"
+		(property "Footprint" "DS_Resistor:R_0402_1005Metric"
 			(at 185.674 147.828 0)
 			(effects
@@
 			)
 		)
-		(property "Footprint" "Capacitor_SMD:C_0402_1005Metric"
+		(property "Footprint" "DS_Capacitor:C_0402_1005Metric"
 			(at 158.75 157.734 0)
 			(show_name yes)
@@
 			)
 		)
-		(property "Footprint" "Resistor_SMD:R_0402_1005Metric"
+		(property "Footprint" "DS_Resistor:R_0402_1005Metric"
 			(at 186.944 70.358 0)
 			(effects
@@
 			)
 		)
-		(property "Footprint" "Resistor_SMD:R_0402_1005Metric"
+		(property "Footprint" "DS_Resistor:R_0402_1005Metric"
 			(at 58.166 78.232 0)
 			(effects
@@
 			)
 		)
-		(property "Footprint" "Capacitor_SMD:C_0402_1005Metric"
+		(property "Footprint" "DS_Capacitor:C_0402_1005Metric"
 			(at 158.75 143.764 0)
 			(show_name yes)
@@
 			)
 		)
-		(property "Footprint" "Resistor_SMD:R_0402_1005Metric"
+		(property "Footprint" "DS_Resistor:R_0402_1005Metric"
 			(at 338.074 219.202 0)
 			(effects
@@
 			)
 		)
-		(property "Footprint" "Resistor_SMD:R_0402_1005Metric"
+		(property "Footprint" "DS_Resistor:R_0402_1005Metric"
 			(at 338.074 78.232 0)
 			(effects
@@
 			)
 		)
-		(property "Footprint" "Resistor_SMD:R_0402_1005Metric"
+		(property "Footprint" "DS_Resistor:R_0402_1005Metric"
 			(at 185.674 155.448 0)
 			(effects
@@
 			)
 		)
-		(property "Footprint" "Capacitor_SMD:C_0402_1005Metric"
+		(property "Footprint" "DS_Capacitor:C_0402_1005Metric"
 			(at 30.48 147.574 0)
 			(show_name yes)

Commit message: minor fixes, start with software
Parts:
- added R94, R95: 100R 1%, DS_Resistor:R_0402_1005Metric, symbol DS_Resistor_0402:100R 1% 0402
Connections:
- net +3.3V: now also IC27.13 (A2); no longer IC24.6 (ADDR_SEL)
- net GND: now also R94.1, R95.1; no longer IC22.6 (ADDR_SEL), IC27.13 (A2)
- net at J19.1 (Pin_1), R91.2: now also D8.3 (A2); no longer D8.4 (A1)
- net at J14.1 (Pin_1), R74.2: now also D6.4 (A1); no longer D6.3 (A2)
- net at J16.1 (Pin_1), R82.2: now also D7.4 (A1); no longer D7.3 (A2)
- net at J18.1 (Pin_1), R90.2: now also D8.4 (A1); no longer D8.3 (A2)
- net at J17.1 (Pin_1), R83.2: now also D7.3 (A2); no longer D7.4 (A1)
- net at J20.1 (Pin_1), R92.2: now also D9.4 (A1); no longer D9.3 (A2)
- net at J21.1 (Pin_1), R93.2: now also D9.3 (A2); no longer D9.4 (A1)
- net at J15.1 (Pin_1), R77.2: now also D6.3 (A2); no longer D6.4 (A1)
- new net: IC24.6 (ADDR_SEL), R95.2
- new net: IC22.6 (ADDR_SEL), R94.2
Other:
- note added: "100R to GND -> Address = 0x4D"
- note added: "Mismatch in datasheet in color. Diodes are swapped"
- note added: "Open -> Address = 0x18"
- note added: "Read expander: A2=1, A1=1, A0=1 -> 0x27"
- note removed: "Read expander: A2=0, A1=1, A0=1 -> 0x23"
- moved on the sheet: D6, D7, D8, D9
